Commit message: arm structure

File: src/first_model.urdf (robot description, URDF)
Before this commit: robot arm, 3 links, 2 joints
Links:
- removed link arm2
- added link actuator1; collision box size=0.04 0.061 0.041; visual box size=0.04 0.061 0.041
- added link actuator2; collision box size=0.031 0.11 0.073; visual box size=0.031 0.11 0.073
- added link connectingbox; collision box size=0.043 0.06 0.0995; visual box size=0.043 0.06 0.0995
- added link tip; collision sphere radius=0.014; visual sphere radius=0.014
- added link tube1; collision cylinder length=0.4 radius=0.014; visual cylinder length=0.4 radius=0.014
- added link tube2; collision cylinder length=0.6 radius=0.02; visual cylinder length=0.6 radius=0.02
- link actuator3: geometry collision box size=0.04 0.061 0.041; visual box size=0.04 0.061 0.041
Joints:
- removed joint actuator_to_tube
- added joint actuator1_to_tube1: type continuous, parent actuator1, child tube1, origin xyz=0 -0.013 0.041, axis 0 0 1
- added joint actuator2_to_tube2: type continuous, parent actuator2, child tube2, origin xyz=-0.031 0 0, axis 1 0 0
- added joint actuator3_to_connectingplate: type continuous, parent actuator3, child connectingbox, origin xyz=0 0.01755 0.041, axis 0 0 1
- added joint connectingbox_to_actuator2: type fixed, parent connectingbox, child actuator2, origin xyz=-0.0215 0 0.06
- added joint tube1_to_tip: type fixed, parent tube1, child tip, origin xyz=0 0.4 0.014
- added joint tube2_to_actuator1: type fixed, parent tube2, child actuator1, origin xyz=0 0.6 0 rpy=0 1.5707963 0
- joint baseplate_to_actuator3: origin xyz=0 0 0 -> xyz=0 0 0.001 rpy=0 0 0

Commit message: updated second model, created first meshes

File: src/first_model.urdf (robot description, URDF)
Before this commit: robot arm, 8 links, 7 joints
Links:
- link tip: geometry collision sphere radius=0.014; visual sphere radius=0.007
- link tube1: geometry collision cylinder length=0.4 radius=0.007; visual cylinder length=0.4 radius=0.007
- link tube2: geometry collision cylinder length=0.6 radius=0.01; visual cylinder length=0.6 radius=0.01
Joints:
- joint tube1_to_tip: origin xyz=0 0.4 0.014 -> xyz=0 0.4 0.007
