Commit message: colors and meshes corrected

File: src/second_model_xacro_version.urdf.xacro (robot description, xacro)
@@ -2,19 +2,26 @@
 <robot name="arm" xmlns:xacro="http://ros.org/wiki/xacro">
   <material name="black">
-    <color rgba="0 0 0 1"/>
+    <color rgba="${0/255} ${0/255} ${0/255} 1.0"/>
+  </material>
+  <material name="dark_grey">
+    <color rgba="${105/255} {105/255} ${105/255} 1.0"/>
+  </material>
+  <material name="grey">
+    <color rgba="${128/255} ${128/255} ${128/255} 1.0"/>
   </material>
   <material name="light_grey">
-    <color rgba="0 0 0 0.2"/>
-  </material>
-  <material name="grey">
-    <color rgba="0 0 0 0.5"/>
-  </material>
-  <material name="dark_grey">
-    <color rgba="0 0 0 0.7"/>
+    <color rgba="${221/255} ${221/255} ${221/255} 1"/>
   </material>
   <material name="white">
-    <color rgba="1 1 1 1"/>
+    <color rgba="${255/255} ${255/255} ${255/255} 1.0"/>
+  </material>
+  <material name="red">
+    <color rgba="${255/255} ${0/255} ${0/255} 1.0"/>
   </material>
   <xacro:property name="pi" value="3.1415269" />
+  <xacro:property name="mesh_scale" value="0.001" />
+  <xacro:property name="mesh_file_tip" value="package://mav_arm_force_controlled/meshes/tip.stl" />
+  <xacro:property name="mesh_file_tube1" value="package://mav_arm_force_controlled/meshes/tube1.stl" />
+  <xacro:property name="mesh_file_actuator1" value="package://mav_arm_force_controlled/meshes/actuator1.stl" />
   <xacro:property name="Baseplate_box_length" value="0.1" />
   <xacro:property name="Baseplate_box_width" value="0.1" />
@@ -98,5 +105,5 @@
       </geometry>
       <origin rpy="0 0 0" xyz="0 0 0.04975"/>
-      <material name="white"/>
+      <material name="dark_grey"/>
     </visual>
     <collision>
@@ -121,5 +128,5 @@
       </geometry>
       <origin rpy="0 0 0" xyz="-0.0155 -0.025 0"/>
-      <material name="white"/>
+      <material name="red"/>
     </visual>
     <collision>
@@ -211,11 +218,12 @@
     <link name="tip">
       <visual>
-        <geometry>
-          <!--
-          <mesh filename="package://mav_arm_force_controlled/meshes/tip.stl"/>
-        -->
+        <!--
           <sphere radius="0.007"/>
-        </geometry>
-        <origin rpy="0 0 0" xyz="0 0 0"/>
+      -->
+      <geometry>
+          <mesh filename="${mesh_file_tip}"
+            scale="${mesh_scale} ${mesh_scale} ${mesh_scale}"/>
+        </geometry>
+        <origin rpy="${-pi/2} 0 0" xyz="0 0 0"/>
         <material name="white"/>
       </visual>

Commit message: ordered

File: src/second_model_xacro_version.urdf.xacro (robot description, xacro)
@@ -1,4 +1,5 @@
 <?xml version="1.0"?>
 <robot name="arm" xmlns:xacro="http://ros.org/wiki/xacro">
+  <!-- Material and Colors-->
   <material name="black">
     <color rgba="${0/255} ${0/255} ${0/255} 1.0"/>
@@ -19,22 +20,26 @@
     <color rgba="${255/255} ${0/255} ${0/255} 1.0"/>
   </material>
-  <xacro:property name="pi" value="3.1415269" />
-  <xacro:property name="mesh_scale" value="0.001" />
-  <xacro:property name="mesh_file_tip" value="package://mav_arm_force_controlled/meshes/tip.stl" />
-  <xacro:property name="mesh_file_tube1" value="package://mav_arm_force_controlled/meshes/tube1.stl" />
-  <xacro:property name="mesh_file_actuator1" value="package://mav_arm_force_controlled/meshes/actuator1.stl" />
-  <xacro:property name="Baseplate_box_length" value="0.1" />
-  <xacro:property name="Baseplate_box_width" value="0.1" />
-  <xacro:property name="Baseplate_box_depth" value="0.001" />
-  <xacro:property name="Baseplate_mass" value="0.040063354" />
-  <xacro:property name="Baseplate_cog_x" value="0.025202079" />
-  <xacro:property name="Baseplate_cog_y" value="0.014500000" />
-  <xacro:property name="Baseplate_cog_z" value="0.000000000" />
-  <xacro:property name="Baseplate_ixx" value="0.000035649" />
-  <xacro:property name="Baseplate_ixy" value="0.000014640" />
-  <xacro:property name="Baseplate_ixz" value="0.000000000" />
-  <xacro:property name="Baseplate_iyy" value="0.000091991" />
-  <xacro:property name="Baseplate_iyz" value="0.000000000" />
-  <xacro:property name="Baseplate_izz" value="0.000073356" />
+    <!-- General Variables-->
+    <xacro:property name="pi" value="3.1415269" />
+    <!-- Mesh files-->
+    <xacro:property name="mesh_file_tip" value="package://mav_arm_force_controlled/meshes/tip.stl" />
+    <xacro:property name="mesh_file_tube1" value="package://mav_arm_force_controlled/meshes/tube1.stl" />
+    <xacro:property name="mesh_file_actuator1" value="package://mav_arm_force_controlled/meshes/actuator1.stl" />
+    <!-- Mesh files are in mm. All mesh files are scaled by the factor 10000-->
+    <xacro:property name="mesh_scale" value="0.001" />
+    <!-- First element, Base Plate-->
+    <xacro:property name="Baseplate_box_length" value="0.1" />
+    <xacro:property name="Baseplate_box_width" value="0.1" />
+    <xacro:property name="Baseplate_box_depth" value="0.001" />
+    <xacro:property name="Baseplate_mass" value="0.040063354" />
+    <xacro:property name="Baseplate_cog_x" value="0.025202079" />
+    <xacro:property name="Baseplate_cog_y" value="0.014500000" />
+    <xacro:property name="Baseplate_cog_z" value="0.000000000" />
+    <xacro:property name="Baseplate_ixx" value="0.000035649" />
+    <xacro:property name="Baseplate_ixy" value="0.000014640" />
+    <xacro:property name="Baseplate_ixz" value="0.000000000" />
+    <xacro:property name="Baseplate_iyy" value="0.000091991" />
+    <xacro:property name="Baseplate_iyz" value="0.000000000" />
+    <xacro:property name="Baseplate_izz" value="0.000073356" />
   <link name="base_plate">
     <visual>
