Commit message: extended inertia of parts

File: src/second_model.urdf.xacro (robot description, xacro)
@@ -28,8 +28,10 @@
     <xacro:property name="mesh_file_hebi" value="package://mav_arm_force_controlled/meshes/hebi.stl" />
     <xacro:property name="mesh_file_hebitotube2" value="package://mav_arm_force_controlled/meshes/hebitotube2.stl" />
-      <!--
-    <xacro:property name="mesh_file_hebhebii" value="package://mav_arm_force_controlled/meshes/hebi.stl" />
-    <xacro:property name="mesh_file_hebi" value="package://mav_arm_force_controlled/meshes/hebi.stl" />
--->
+    <xacro:property name="mesh_file_mesh_file_tube2" value="package://mav_arm_force_controlled/meshes/mesh_file_tube2.stl" />
+    <xacro:property name="mesh_file_mesh_file_clamp2" value="package://mav_arm_force_controlled/meshes/mesh_file_clamp2.stl" />
+    <xacro:property name="mesh_file_mesh_file_actuator1" value="package://mav_arm_force_controlled/meshes/mesh_file_actuator1.stl" />
+    <xacro:property name="mesh_file_mesh_file_clamp1" value="package://mav_arm_force_controlled/meshes/mesh_file_clamp1.stl" />
+    <xacro:property name="mesh_file_mesh_file_tube1" value="package://mav_arm_force_controlled/meshes/mesh_file_tube1.stl" />
+    <xacro:property name="mesh_file_mesh_file_tip" value="package://mav_arm_force_controlled/meshes/mesh_file_tip.stl" />
     <!-- Mesh files are in mm. All mesh files are scaled by the factor 10000-->
     <xacro:property name="mesh_scale" value="0.001" />
@@ -90,4 +92,6 @@
     <collision>
       <geometry>
+        <mesh filename="${mesh_file_dyamixel}"
+              scale="${mesh_scale} ${mesh_scale} ${mesh_scale}"/>
       </geometry>
     </collision>
@@ -135,6 +139,16 @@
     <parent link="connectingbox"/>
     <child link="actuator2"/>
-    <origin rpy="${pi/2} ${0} ${pi/2}"  xyz="${0.025} ${0} ${0.001+0.055}"/>
-  </joint>
+    <origin rpy="${pi/2} ${0} ${pi/2}"  xyz="${0.005+0.015} ${0} ${0.055}"/>
+  </joint>
+  <xacro:property name="actuator2_mass" value=" 0.34" />
+  <xacro:property name="actuator2_cog_x" value="0.000000171" />
+  <xacro:property name="actuator2_cog_y" value="0.000278026" />
+  <xacro:property name="actuator2_cog_z" value="0.038471524" />
+  <xacro:property name="actuator2_ixx" value="0.000186786" />
+  <xacro:property name="actuator2_ixy" value="0.000041556" />
+  <xacro:property name="actuator2_ixz" value="0.000000273" />
+  <xacro:property name="actuator2_iyy" value="0.00043422" />
+  <xacro:property name="actuator2_iyz" value="0.00000029" />
+  <xacro:property name="actuator2_izz" value="0.000554524" />
   <link name="actuator2">
     <visual>
@@ -152,6 +166,6 @@
     </collision>
     <inertia>
-      <mass value="0.34"/>
-      <inertia ixx="0.001" ixy="0" ixz="0" iyy="0.001" iyz="0" izz="0.001" />
+      <mass value="actuator2_mass"/>
+      <inertia ixx="{actuator2_ixx}" ixy="${actuator2_ixy}" ixz="${actuator2_ixz}" iyy="${actuator2_iyy}" iyz="${actuator2_iyz}" izz="${actuator2_izz}" />
     </inertia>
   </link>
@@ -160,6 +174,16 @@
     <parent link="actuator2"/>
     <child link="clamp3"/>
-    <origin rpy="0 0 0" xyz="${0} 0 ${0.01605}"/>
-  </joint>
+    <origin rpy="${pi/2} 0 ${-pi/2}" xyz="${0} 0 ${0.01605}"/>
+  </joint>
+  <xacro:property name="clamp3_mass" value=" 0." />
+  <xacro:property name="clamp3_cog_x" value="0.015022968" />
+  <xacro:property name="clamp3_cog_y" value="0.001776283" />
+  <xacro:property name="clamp3_cog_z" value="0.000017898" />
+  <xacro:property name="clamp3_ixx" value="0.000524947" />
+  <xacro:property name="clamp3_ixy" value="0.000000017" />
+  <xacro:property name="clamp3_ixz" value="-0.00000004" />
+  <xacro:property name="clamp3_iyy" value="0.000535726" />
+  <xacro:property name="clamp3_iyz" value="-0.000092479" />
+  <xacro:property name="clamp3_izz" value="0.000074342" />
   <link name="clamp3">
     <visual>
@@ -177,30 +201,39 @@
     </collision>
     <inertia>
-      <mass value="0.01"/>
-      <inertia ixx="0.000917686" ixy="0.000000017" ixz="0.000000018" iyy="0.000928465" iyz="0.000093232" izz="0.000074342" />
-    </inertia>
-  </link>
-    <!--
+      <mass value="clamp3_mass"/>
+      <inertia ixx="clamp3_ixx" ixy="clamp3_ixy" ixz="clamp3_ixz" iyy="clamp3_iyy" iyz="clamp3_iyz" izz="clamp3_izz" />
+    </inertia>
+  </link>
   <joint name="clamp3_to_tube2" type="fixed">
     <parent link="clamp3"/>
     <child link="tube2"/>
-    <origin xyz="-0.031 0 0"/>
-  </joint>
+    <origin xyz="0 0.05 0"/>
+  </joint>
+  <xacro:property name="tube2_mass" value="" />
+  <xacro:property name="tube2_cog_x" value="" />
+  <xacro:property name="tube2_cog_y" value="" />
+  <xacro:property name="tube2_cog_z" value="" />
+  <xacro:property name="tube2_ixx" value="" />
+  <xacro:property name="tube2_ixy" value="" />
+  <xacro:property name="tube2_ixz" value="" />
+  <xacro:property name="tube2_iyy" value="" />
+  <xacro:property name="tube2_iyz" value="" />
+  <xacro:property name="tube2_izz" value="" />
   <link name="tube2">
     <visual>
       <geometry>
-        <cylinder length="0.6" radius="0.01"/>
-      </geometry>
-      <origin rpy="1.570796 0 0" xyz="-0.01 0.3 0"/>
-      <material name="light_grey"/>
-    </visual>
-    <collision>
-      <geometry>
-        <cylinder length="0.6" radius="0.01"/>
-      </geometry>
-    </collision>
-    <inertia>
-      <mass value="0.01"/>
-      <inertia ixx="0.0012" ixy="0" ixz="0" iyy="0" iyz="0" izz="0.0012" />
+        <mesh filename="${mesh_file_tube2}"
+              scale="${mesh_scale} ${mesh_scale} ${mesh_scale}"/>
+      </geometry>
+      <origin rpy="0 0 0" xyz="0 0 0"/>
+      <material name="red"/>
+    </visual>
+    <collision>
+      <geometry>
+      </geometry>
+    </collision>
+    <inertia>
+      <mass value="tube2_mass"/>
+      <inertia ixx="tube2_ixx" ixy="tube2_ixy" ixz="tube2_ixz" iyy="tube2_iyy" iyz="tube2_iyz" izz="tube2_izz" />
     </inertia>
   </link>
@@ -210,20 +243,30 @@
       <origin rpy="0 0 0" xyz="0 0.3 0"/>
     </joint>
+    <xacro:property name="clamp2_mass" value="" />
+    <xacro:property name="clamp2_cog_x" value="" />
+    <xacro:property name="clamp2_cog_y" value="" />
+    <xacro:property name="clamp2_cog_z" value="" />
+    <xacro:property name="clamp2_ixx" value="" />
+    <xacro:property name="clamp2_ixy" value="" />
+    <xacro:property name="clamp2_ixz" value="" />
+    <xacro:property name="clamp2_iyy" value="" />
+    <xacro:property name="clamp2_iyz" value="" />
+    <xacro:property name="clamp2_izz" value="" />
     <link name="clamp2">
       <visual>
         <geometry>
-          <sphere radius="0.02"/>
-        </geometry>
-        <origin rpy="1.570796 0 0" xyz="-0.01 0.3 0"/>
+          <mesh filename="${mesh_file_clamp2}"
+                scale="${mesh_scale} ${mesh_scale} ${mesh_scale}"/>
+        </geometry>
+        <origin rpy="0 0 0" xyz="-0.01 0.3 0"/>
         <material name="black"/>
       </visual>
       <collision>
         <geometry>
-          <sphere radius="0.02"/>
         </geometry>
       </collision>
       <inertia>
-        <mass value="0.01"/>
-        <inertia ixx="0.0012" ixy="0" ixz="0" iyy="0" iyz="0" izz="0.0012" />
+        <mass value="clamp2_mass"/>
+        <inertia ixx="clamp2_ixx" ixy="clamp2_ixy" ixz="clamp2_ixz" iyy="clamp2_iyy" iyz="clamp2_iyz" izz="clamp2_izz" />
       </inertia>
     </link>
@@ -231,12 +274,56 @@
         <parent link="clamp2"/>
         <child link="actuator1"/>
-        <origin rpy="0 1.5707963 0" xyz="0 0.3 0"/>
+        <origin rpy="0 0 0" xyz="0 0.3 0"/>
       </joint>
-  <link name="actuator1">
-    <visual>
-      <geometry>
-          <mesh filename="${mesh_file_actuator1}"
-            scale="${mesh_scale} ${mesh_scale} ${mesh_scale}"/>
-        </geometry>
+      <xacro:property name="actuator1_mass" value="" />
+      <xacro:property name="actuator1_cog_x" value="" />
+      <xacro:property name="actuator1_cog_y" value="" />
+      <xacro:property name="actuator1_cog_z" value="" />
+      <xacro:property name="actuator1_ixx" value="" />
+      <xacro:property name="actuator1_ixy" value="" />
+      <xacro:property name="actuator1_ixz" value="" />
+      <xacro:property name="actuator1_iyy" value="" />
+      <xacro:property name="actuator1_iyz" value="" />
+      <xacro:property name="actuator1_izz" value="" />
+    <link name="actuator1">
+      <visual>
+        <geometry>
+            <mesh filename="${mesh_file_actuator1}"
+              scale="${mesh_scale} ${mesh_scale} ${mesh_scale}"/>
+          </geometry>
+        <origin rpy="0 0 0" xyz="0 0 0"/>
+        <material name="black"/>
+      </visual>
+      <collision>
+        <geometry>
+        </geometry>
+      </collision>
+      <inertia>
+        <mass value="actuator1_mass"/>
+        <inertia ixx="actuator1_ixx" ixy="actuator1_ixy" ixz="actuator1_ixz" iyy="actuator1_iyy" iyz="actuator1_iyz" izz="actuator1_izz" />
+      </inertia>
+    </link>
+  <joint name="actuator1_to_clamp1" type="continuous">
+    <axis rpy="0 0 0" xyz="0 0 0"/>
+    <parent link="actuator1"/>
+    <child link="clamp1"/>
+    <origin xyz="0 0 0"/>
+  </joint>
+  <xacro:property name="clamp1_mass" value="" />
+  <xacro:property name="clamp1_cog_x" value="" />
+  <xacro:property name="clamp1_cog_y" value="" />
+  <xacro:property name="clamp1_cog_z" value="" />
+  <xacro:property name="clamp1_ixx" value="" />
+  <xacro:property name="clamp1_ixy" value="" />
+  <xacro:property name="clamp1_ixz" value="" />
+  <xacro:property name="clamp1_iyy" value="" />
+  <xacro:property name="clamp1_iyz" value="" />
+  <xacro:property name="clamp1_izz" value="" />
+  <link name="clamp1">
+    <visual>
+      <geometry>
+        <mesh filename="${mesh_file_clamp1}"
+          scale="${mesh_scale} ${mesh_scale} ${mesh_scale}"/>
+      </geometry>
       <origin rpy="0 0 0" xyz="0 -0.0305 0.0205"/>
       <material name="black"/>
@@ -244,34 +331,9 @@
     <collision>
       <geometry>
-        <box size="0.04 0.061 0.041"/>
-      </geometry>
-    </collision>
-    <inertia>
-      <mass value="0.22"/>
-      <inertia ixx="0.00003691125" ixy="0" ixz="0" iyy="0.00005986125" iyz="0" izz="0.0000607725" />
-    </inertia>
-  </link>
-  <joint name="actuator1_to_clamp1" type="continuous">
-    <axis rpy="0 0 0" xyz="0 0 1"/>
-    <parent link="actuator1"/>
-    <child link="clamp1"/>
-    <origin xyz="0 -0.013 0.041"/>
-  </joint>
-  <link name="clamp1">
-    <visual>
-      <geometry>
-        <sphere radius="0.02"/>
-      </geometry>
-      <origin rpy="0 0 0" xyz="0 -0.0305 0.0205"/>
-      <material name="black"/>
-    </visual>
-    <collision>
-      <geometry>
-        <sphere radius="0.02"/>
-      </geometry>
-    </collision>
-    <inertia>
-      <mass value="0.22"/>
-      <inertia ixx="0.00003691125" ixy="0" ixz="0" iyy="0.00005986125" iyz="0" izz="0.0000607725" />
+      </geometry>
+    </collision>
+    <inertia>
+      <mass value="clamp1_mass"/>
+      <inertia ixx="clamp1_ixx" ixy="clamp1_ixy" ixz="clamp1_ixz" iyy="clamp1_iyy" iyz="clamp1_iyz" izz="clamp1_izz" />
     </inertia>
   </link>
@@ -281,20 +343,30 @@
     <origin xyz="0 0 0"/>
   </joint>
+  <xacro:property name="tube1_mass" value="" />
+  <xacro:property name="tube1_cog_x" value="" />
+  <xacro:property name="tube1_cog_y" value="" />
+  <xacro:property name="tube1_cog_z" value="" />
+  <xacro:property name="tube1_ixx" value="" />
+  <xacro:property name="tube1_ixy" value="" />
+  <xacro:property name="tube1_ixz" value="" />
+  <xacro:property name="tube1_iyy" value="" />
+  <xacro:property name="tube1_iyz" value="" />
+  <xacro:property name="tube1_izz" value="" />
     <link name="tube1">
       <visual>
         <geometry>
-          <cylinder length="0.4" radius="0.007"/>
-        </geometry>
-        <origin rpy="1.570796 0 0" xyz="0 0.2 0.007"/>
-        <material name="light_grey"/>
+          <mesh filename="${mesh_file_tube1}"
+            scale="${mesh_scale} ${mesh_scale} ${mesh_scale}"/>
+        </geometry>
+        <origin rpy="0 0 0" xyz="0 0 0"/>
+        <material name="dark_grey"/>
       </visual>
       <collision>
         <geometry>
-          <cylinder length="0.4" radius="0.007"/>
         </geometry>
       </collision>
       <inertia>
-        <mass value="0.01"/>
-        <inertia ixx="0.0012" ixy="0" ixz="0" iyy="0" iyz="0" izz="0.0012" />
+        <mass value="tube1_mass"/>
+        <inertia ixx="tube1_ixx" ixy="tube1_ixy" ixz="tube1_ixz" iyy="tube1_iyy" iyz="tube1_iyz" izz="tube1_izz" />
       </inertia>
     </link>
@@ -304,4 +376,14 @@
       <origin xyz="0 0.4 0.007"/>
     </joint>
+    <xacro:property name="tip_mass" value="" />
+    <xacro:property name="tip_cog_x" value="" />
+    <xacro:property name="tip_cog_y" value="" />
+    <xacro:property name="tip_cog_z" value="" />
+    <xacro:property name="tip_ixx" value="" />
+    <xacro:property name="tip_ixy" value="" />
+    <xacro:property name="tip_ixz" value="" />
+    <xacro:property name="tip_iyy" value="" />
+    <xacro:property name="tip_iyz" value="" />
+    <xacro:property name="tip_izz" value="" />
     <link name="tip">
       <visual>
@@ -310,17 +392,15 @@
             scale="${mesh_scale} ${mesh_scale} ${mesh_scale}"/>
         </geometry>
-        <origin rpy="${-pi/2} 0 0" xyz="0 0 0"/>
+        <origin rpy="0 0 0" xyz="0 0 0"/>
         <material name="white"/>
       </visual>
       <collision>
         <geometry>
-          <sphere radius="0.014"/>
         </geometry>
       </collision>
       <inertia>
-        <mass value="0.01"/>
-        <inertia ixx="0.00028" ixy="0" ixz="0" iyy="0.00028" iyz="0" izz="0.00028" />
+        <mass value="tip_mass"/>
+        <inertia ixx="tip_ixx" ixy="tip_ixy" ixz="tip_ixz" iyy="tip_iyy" iyz="tip_iyz" izz="tip_izz" />
       </inertia>
     </link>
--->
 </robot>
