Commit message: fixed some xacro inertia syntax

File: src/thirdmodel.urdf.xacro (robot description, xacro)
@@ -137,5 +137,5 @@
     <origin rpy="${pi/2} ${0} ${pi/2}"  xyz="${0.005+0.015} ${0} ${0.0635}"/>
   </joint>
-  <xacro:property name="actuator2_mass" value=" 0.34" />
+  <xacro:property name="actuator2_mass" value="0.34" />
   <xacro:property name="actuator2_cog_x" value="0.000000171" />
   <xacro:property name="actuator2_cog_y" value="0.000278026" />
@@ -158,9 +158,9 @@
     <inertia>
       <mass value="actuator2_mass"/>
-      <inertia ixx="{actuator2_ixx}" ixy="${actuator2_ixy}" ixz="${actuator2_ixz}" iyy="${actuator2_iyy}" iyz="${actuator2_iyz}" izz="${actuator2_izz}" />
+      <inertia ixx="${actuator2_ixx}" ixy="${actuator2_ixy}" ixz="${actuator2_ixz}" iyy="${actuator2_iyy}" iyz="${actuator2_iyz}" izz="${actuator2_izz}" />
     </inertia>
   </link>
   <joint name="actuator2_to_clamp3" type="continuous">
-    <axis rpy="0 0 0" xyz="0 1 0"/> />
+    <axis rpy="0 0 0" xyz="0 1 0"/>
     <parent link="actuator2"/>
     <child link="clamp3"/>
@@ -177,5 +177,5 @@
     </joint>
   </transmission>
-  <xacro:property name="clamp3_mass" value=" 0." />
+  <xacro:property name="clamp3_mass" value="0.21" />
   <xacro:property name="clamp3_cog_x" value="0.015022968" />
   <xacro:property name="clamp3_cog_y" value="0.001776283" />
@@ -202,6 +202,6 @@
     </collision>
     <inertia>
-      <mass value="clamp3_mass"/>
-      <inertia ixx="clamp3_ixx" ixy="clamp3_ixy" ixz="clamp3_ixz" iyy="clamp3_iyy" iyz="clamp3_iyz" izz="clamp3_izz" />
+      <mass value="${clamp3_mass}"/>
+      <inertia ixx="${clamp3_ixx}" ixy="${clamp3_ixy}" ixz="${clamp3_ixz}" iyy="${clamp3_iyy}" iyz="${clamp3_iyz}" izz="${clamp3_izz}" />
     </inertia>
   </link>
@@ -232,5 +232,5 @@
     <inertia>
       <mass value="tube2_mass"/>
-      <inertia ixx="tube2_ixx" ixy="tube2_ixy" ixz="tube2_ixz" iyy="tube2_iyy" iyz="tube2_iyz" izz="tube2_izz" />
+      <inertia ixx="${tube2_ixx}" ixy="${tube2_ixy}" ixz="${tube2_ixz}" iyy="${tube2_iyy}" iyz="${tube2_iyz}" izz="${tube2_izz}" />
     </inertia>
   </link>
@@ -261,5 +261,5 @@
       <inertia>
         <mass value="clamp2_mass"/>
-        <inertia ixx="clamp2_ixx" ixy="clamp2_ixy" ixz="clamp2_ixz" iyy="clamp2_iyy" iyz="clamp2_iyz" izz="clamp2_izz" />
+        <inertia ixx="${clamp2_ixx}" ixy="${clamp2_ixy}" ixz="${clamp2_ixz}" iyy="${clamp2_iyy}" iyz="${clamp2_iyz}" izz="${clamp2_izz}" />
       </inertia>
     </link>
@@ -290,5 +290,5 @@
       <inertia>
         <mass value="actuator1_mass"/>
-        <inertia ixx="actuator1_ixx" ixy="actuator1_ixy" ixz="actuator1_ixz" iyy="actuator1_iyy" iyz="actuator1_iyz" izz="actuator1_izz" />
+        <inertia ixx="${actuator1_ixx}" ixy="${actuator1_ixy}" ixz="${actuator1_ixz}" iyy="${actuator1_iyy}" iyz="${actuator1_iyz}" izz="${actuator1_izz}" />
       </inertia>
     </link>
@@ -330,5 +330,5 @@
     <inertia>
       <mass value="clamp1_mass"/>
-      <inertia ixx="clamp1_ixx" ixy="clamp1_ixy" ixz="clamp1_ixz" iyy="clamp1_iyy" iyz="clamp1_iyz" izz="clamp1_izz" />
+      <inertia ixx="${clamp1_ixx}" ixy="${clamp1_ixy}" ixz="${clamp1_ixz}" iyy="${clamp1_iyy}" iyz="${clamp1_iyz}" izz="${clamp1_izz}" />
     </inertia>
   </link>
@@ -359,5 +359,5 @@
       <inertia>
         <mass value="tube1_mass"/>
-        <inertia ixx="tube1_ixx" ixy="tube1_ixy" ixz="tube1_ixz" iyy="tube1_iyy" iyz="tube1_iyz" izz="tube1_izz" />
+        <inertia ixx="${tube1_ixx}" ixy="${tube1_ixy}" ixz="${tube1_ixz}" iyy="${tube1_iyy}" iyz="${tube1_iyz}" izz="${tube1_izz}" />
       </inertia>
     </link>
@@ -388,5 +388,5 @@
       <inertia>
         <mass value="tip_mass"/>
-        <inertia ixx="tip_ixx" ixy="tip_ixy" ixz="tip_ixz" iyy="tip_iyy" iyz="tip_iyz" izz="tip_izz" />
+        <inertia ixx="${tip_ixx}" ixy="${tip_ixy}" ixz="${tip_ixz}" iyy="${tip_iyy}" iyz="${tip_iyz}" izz="${tip_izz}" />
       </inertia>
     </link>

Commit message: first successful gazebo run

File: src/thirdmodel.urdf.xacro (robot description, xacro)
@@ -3,11 +3,11 @@
   <!-- Material and Colors-->
   <material name="black">
-    <color rgba="${0/255} ${0/255} ${0/255} 1.0"/>
+    <color rgba="${0/255} ${0/255} ${0/255} 1"/>
   </material>
   <material name="dark_grey">
-    <color rgba="${105/255} {105/255} ${105/255} 1.0"/>
+    <color rgba="${105/255} ${105/255} ${105/255} 1"/>
   </material>
   <material name="grey">
-    <color rgba="${128/255} ${128/255} ${128/255} 1.0"/>
+    <color rgba="${128/255} ${128/255} ${128/255} 1"/>
   </material>
   <material name="light_grey">
@@ -15,8 +15,8 @@
   </material>
   <material name="white">
-    <color rgba="${255/255} ${255/255} ${255/255} 1.0"/>
+    <color rgba="${255/255} ${255/255} ${255/255} 1"/>
   </material>
   <material name="red">
-    <color rgba="${255/255} ${0/255} ${0/255} 1.0"/>
+    <color rgba="${255/255} ${0/255} ${0/255} 1"/>
   </material>
     <!-- General Variables-->
@@ -57,8 +57,14 @@
       <material name="black"/>
     </visual>
-    <inertia>
+    <collision>
+      <geometry>
+        <box size="0.1 0.1 0.1"/>
+        </geometry>
+      <origin rpy="0 0 0" xyz="0 0 0"/>
+    </collision>
+    <inertial>
       <mass value="${baseplate_mass}"/>
       <inertia ixx="${baseplate_ixx}" ixy="${baseplate_ixy}" ixz="${baseplate_ixz}" iyy="${baseplate_iyy}" iyz="${baseplate_iyz}" izz="${baseplate_izz}" />
-    </inertia>
+    </inertial>
   </link>
   <joint name="baseplate_to_actuator3" type="fixed">
@@ -86,11 +92,16 @@
         <material name="black"/>
     </visual>
-    <inertia>
-      <origin xyz="dynamixel_cog_x dynamixel_cog_y dynamixel_cog_z"/>
+    <collision>
+      <geometry>
+        <box size="0.1 0.1 0.1"/>
+        </geometry>
+      <origin rpy="0 0 0" xyz="0 0 0"/>
+    </collision>
+    <inertial>
       <mass value="${dynamixel_mass}"/>
       <inertia ixx="${dynamixel_ixy}" ixy="${dynamixel_ixy}" ixz="${dynamixel_ixz}" iyy="${dynamixel_iyy}" iyz="${dynamixel_iyz}" izz="${dynamixel_izz}" />
-    </inertia>
-  </link>
-  <joint name="actuator3_to_connectingplate" type="continuous">
+    </inertial>
+  </link>
+  <joint name="actuator_to_connectingbox" type="continuous">
     <axis rpy="0 0 0" xyz="0 0 1"/>
     <parent link="actuator3"/>
@@ -99,10 +110,10 @@
     <limit effort="30" velocity="1.0"/>
   </joint>
-  <transmission name="actuator3_dynamixel">
+  <transmission name="actuator3_dynamixel_trans">
     <type>transmission_interface/SimpleTransmission</type>
-    <actuator name="$actuator3_dynamixel">
+    <actuator name="actuator3_dynamixel_a">
       <mechanicalReduction>1</mechanicalReduction>
     </actuator>
-    <joint name="actuator3_to_connectingplate">
+    <joint name="actuator_to_connectingbox">
       <hardwareInterface>PositionJointInterface</hardwareInterface>
     </joint>
@@ -127,8 +138,14 @@
       <material name="black"/>
     </visual>
-    <inertia>
-      <mass value="0.01"/>
+    <collision>
+      <geometry>
+        <box size="0.1 0.1 0.1"/>
+        </geometry>
+      <origin rpy="0 0 0" xyz="0 0 0"/>
+    </collision>
+    <inertial>
+      <mass value="${connectionmx64hebi_mass}"/>
       <inertia ixx="${connectionmx64hebi_ixx}" ixy="${connectionmx64hebi_ixy}" ixz="${connectionmx64hebi_ixz}" iyy="${connectionmx64hebi_iyy}" iyz="${connectionmx64hebi_iyz}" izz="${connectionmx64hebi_izz}" />
-    </inertia>
+    </inertial>
   </link>
   <joint name="connectingbox_to_actuator2" type="fixed">
@@ -156,8 +173,14 @@
       <material name="red"/>
     </visual>
-    <inertia>
-      <mass value="actuator2_mass"/>
+    <collision>
+      <geometry>
+        <box size="0.1 0.1 0.1"/>
+        </geometry>
+      <origin rpy="0 0 0" xyz="0 0 0"/>
+    </collision>
+    <inertial>
+      <mass value="${actuator2_mass}"/>
       <inertia ixx="${actuator2_ixx}" ixy="${actuator2_ixy}" ixz="${actuator2_ixz}" iyy="${actuator2_iyy}" iyz="${actuator2_iyz}" izz="${actuator2_izz}" />
-    </inertia>
+    </inertial>
   </link>
   <joint name="actuator2_to_clamp3" type="continuous">
@@ -168,5 +191,5 @@
     <limit effort="30" velocity="1.0"/>
   </joint>
-  <transmission name="actuator2_hebi">
+  <!-- <transmission name="actuator2_hebi">
     <type>transmission_interface/SimpleTransmission</type>
     <actuator name="$actuator2_hebi">
@@ -176,5 +199,5 @@
       <hardwareInterface>PositionJointInterface</hardwareInterface>
     </joint>
-  </transmission>
+  </transmission> -->
   <xacro:property name="clamp3_mass" value="0.21" />
   <xacro:property name="clamp3_cog_x" value="0.015022968" />
@@ -198,11 +221,12 @@
     <collision>
       <geometry>
-        <sphere radius="0.02"/>
-      </geometry>
-    </collision>
-    <inertia>
+        <box size="0.1 0.1 0.1"/>
+        </geometry>
+      <origin rpy="0 0 0" xyz="0 0 0"/>
+    </collision>
+    <inertial>
       <mass value="${clamp3_mass}"/>
       <inertia ixx="${clamp3_ixx}" ixy="${clamp3_ixy}" ixz="${clamp3_ixz}" iyy="${clamp3_iyy}" iyz="${clamp3_iyz}" izz="${clamp3_izz}" />
-    </inertia>
+    </inertial>
   </link>
   <joint name="clamp3_to_tube2" type="fixed">
@@ -230,8 +254,14 @@
       <material name="red"/>
     </visual>
-    <inertia>
-      <mass value="tube2_mass"/>
+    <collision>
+      <geometry>
+        <box size="0.1 0.1 0.1"/>
+        </geometry>
+      <origin rpy="0 0 0" xyz="0 0 0"/>
+    </collision>
+    <inertial>
+      <mass value="${tube2_mass}"/>
       <inertia ixx="${tube2_ixx}" ixy="${tube2_ixy}" ixz="${tube2_ixz}" iyy="${tube2_iyy}" iyz="${tube2_iyz}" izz="${tube2_izz}" />
-    </inertia>
+    </inertial>
   </link>
     <joint name="tube2_to_clamp2" type="fixed">
@@ -259,8 +289,14 @@
         <material name="black"/>
       </visual>
-      <inertia>
-        <mass value="clamp2_mass"/>
+      <collision>
+        <geometry>
+          <box size="0.1 0.1 0.1"/>
+          </geometry>
+        <origin rpy="0 0 0" xyz="0 0 0"/>
+      </collision>
+      <inertial>
+        <mass value="${clamp2_mass}"/>
         <inertia ixx="${clamp2_ixx}" ixy="${clamp2_ixy}" ixz="${clamp2_ixz}" iyy="${clamp2_iyy}" iyz="${clamp2_iyz}" izz="${clamp2_izz}" />
-      </inertia>
+      </inertial>
     </link>
       <joint name="clamp2_to_actuator1" type="fixed">
@@ -288,8 +324,14 @@
         <material name="black"/>
       </visual>
-      <inertia>
-        <mass value="actuator1_mass"/>
+      <collision>
+        <geometry>
+          <box size="0.1 0.1 0.1"/>
+          </geometry>
+        <origin rpy="0 0 0" xyz="0 0 0"/>
+      </collision>
+      <inertial>
+        <mass value="${actuator1_mass}"/>
         <inertia ixx="${actuator1_ixx}" ixy="${actuator1_ixy}" ixz="${actuator1_ixz}" iyy="${actuator1_iyy}" iyz="${actuator1_iyz}" izz="${actuator1_izz}" />
-      </inertia>
+      </inertial>
     </link>
   <joint name="actuator1_to_clamp1" type="continuous">
@@ -300,5 +342,5 @@
     <limit effort="30" velocity="1.0"/>
   </joint>
-  <transmission name="actuator1_dynamixel">
+  <!-- <transmission name="actuator1_dynamixel">
     <type>transmission_interface/SimpleTransmission</type>
     <actuator name="$actuator1_dynamixel">
@@ -308,5 +350,5 @@
       <hardwareInterface>PositionJointInterface</hardwareInterface>
     </joint>
-  </transmission>
+  </transmission> -->
   <xacro:property name="clamp1_mass" value="0.11739877" />
   <xacro:property name="clamp1_cog_x" value="0.008717092" />
@@ -328,8 +370,14 @@
       <material name="red"/>
     </visual>
-    <inertia>
-      <mass value="clamp1_mass"/>
+    <collision>
+      <geometry>
+        <box size="0.1 0.1 0.1"/>
+        </geometry>
+      <origin rpy="0 0 0" xyz="0 0 0"/>
+    </collision>
+    <inertial>
+      <mass value="${clamp1_mass}"/>
       <inertia ixx="${clamp1_ixx}" ixy="${clamp1_ixy}" ixz="${clamp1_ixz}" iyy="${clamp1_iyy}" iyz="${clamp1_iyz}" izz="${clamp1_izz}" />
-    </inertia>
+    </inertial>
   </link>
   <joint name="clamp1_to_tube1" type="fixed">
@@ -357,8 +405,14 @@
         <material name="black"/>
       </visual>
-      <inertia>
-        <mass value="tube1_mass"/>
+      <collision>
+        <geometry>
+          <box size="0.1 0.1 0.1"/>
+          </geometry>
+        <origin rpy="0 0 0" xyz="0 0 0"/>
+      </collision>
+      <inertial>
+        <mass value="${tube1_mass}"/>
         <inertia ixx="${tube1_ixx}" ixy="${tube1_ixy}" ixz="${tube1_ixz}" iyy="${tube1_iyy}" iyz="${tube1_iyz}" izz="${tube1_izz}" />
-      </inertia>
+      </inertial>
     </link>
     <joint name="tube1_to_tip" type="fixed">
@@ -386,8 +440,14 @@
         <material name="white"/>
       </visual>
-      <inertia>
-        <mass value="tip_mass"/>
+      <collision>
+        <geometry>
+          <box size="0.1 0.1 0.1"/>
+          </geometry>
+        <origin rpy="0 0 0" xyz="0 0 0"/>
+      </collision>
+      <inertial>
+        <mass value="${tip_mass}"/>
         <inertia ixx="${tip_ixx}" ixy="${tip_ixy}" ixz="${tip_ixz}" iyy="${tip_iyy}" iyz="${tip_iyz}" izz="${tip_izz}" />
-      </inertia>
+      </inertial>
     </link>
     <gazebo>

Commit message: gazebo and roscontrol

File: src/thirdmodel.urdf.xacro (robot description, xacro)
@@ -54,6 +54,5 @@
         </geometry>
       <origin rpy="0 0 0" xyz="0 0 0"/>
-      <!--<origin rpy="0 0 0" xyz="${Baseplate_cog_x} ${Baseplate_cog_y} ${Baseplate_cog_z}"/>-->
-      <material name="black"/>
+       <material name="black"/>
     </visual>
     <collision>

Commit message: corrected namespace and transmissions

File: src/thirdmodel.urdf.xacro (robot description, xacro)
@@ -47,4 +47,10 @@
     <xacro:property name="baseplate_iyz" value="0" />
     <xacro:property name="baseplate_izz" value="0.000214186" />
+  <link name="world"/>
+  <joint name="fixed" type="fixed">
+    <parent link="world"/>
+    <child link="baseplate"/>
+    <origin xyz="0.5 0.5 0" rpy="0 0 0" />
+  </joint>
   <link name="baseplate">
     <visual>
@@ -115,5 +121,5 @@
     </actuator>
     <joint name="actuator_to_connectingbox">
-      <hardwareInterface>PositionJointInterface</hardwareInterface>
+      <hardwareInterface>hardware_interface/EffortJointInterface</hardwareInterface>
     </joint>
   </transmission>
@@ -196,5 +202,5 @@
     </actuator>
     <joint name="actuator2_to_clamp3">
-      <hardwareInterface>PositionJointInterface</hardwareInterface>
+      <hardwareInterface>hardware_interface/EffortJointInterface</hardwareInterface>
     </joint>
   </transmission>
@@ -347,5 +353,5 @@
     </actuator>
     <joint name="actuator1_to_clamp1">
-      <hardwareInterface>PositionJointInterface</hardwareInterface>
+      <hardwareInterface>hardware_interface/EffortJointInterface</hardwareInterface>
     </joint>
   </transmission>
@@ -452,6 +458,7 @@
     <gazebo>
       <plugin name="gazebo_ros_control" filename="libgazebo_ros_control.so">
-        <robotNamespace>/</robotNamespace>
+        <robotNamespace>/arm</robotNamespace>
       </plugin>
     </gazebo>
+        <!--<robotSimType>gazebo_ros_control/DefaultRobotHWSim</robotSimType>-->
 </robot>

Commit message: added simplified meshes for collision checking

File: src/thirdmodel.urdf.xacro (robot description, xacro)
@@ -22,16 +22,28 @@
     <!-- General Variables-->
     <xacro:property name="pi" value="3.1415269" />
-    <!-- Mesh files-->
-    <xacro:property name="mesh_file_baseplate" value="package://mav_arm_force_controlled/meshes/baseplate.stl" />
-    <xacro:property name="mesh_file_dyamixel" value="package://mav_arm_force_controlled/meshes/dynamixel.stl" />
-    <xacro:property name="mesh_file_connecting" value="package://mav_arm_force_controlled/meshes/connecting.stl" />
-    <xacro:property name="mesh_file_hebi" value="package://mav_arm_force_controlled/meshes/hebi.stl" />
-    <xacro:property name="mesh_file_hebitotube2" value="package://mav_arm_force_controlled/meshes/hebitotube2.stl" />
-    <xacro:property name="mesh_file_tube2" value="package://mav_arm_force_controlled/meshes/tube2.stl" />
-    <xacro:property name="mesh_file_clamp2" value="package://mav_arm_force_controlled/meshes/tube2todynamixel.stl" />
-    <xacro:property name="mesh_file_actuator1" value="package://mav_arm_force_controlled/meshes/dynamixel.stl" />
-    <xacro:property name="mesh_file_clamp1" value="package://mav_arm_force_controlled/meshes/dynamixeltotube1.stl" />
-    <xacro:property name="mesh_file_tube1" value="package://mav_arm_force_controlled/meshes/tube1.stl" />
-    <xacro:property name="mesh_file_tip" value="package://mav_arm_force_controlled/meshes/tip.stl" />
+    <!-- Mesh files of exact geometry-->
+    <xacro:property name="mesh_file_baseplate" value="package://mav_arm_force_controlled/meshes/geometry/baseplate.stl" />
+    <xacro:property name="mesh_file_dyamixel" value="package://mav_arm_force_controlled/meshes/geometry/dynamixel.stl" />
+    <xacro:property name="mesh_file_connecting" value="package://mav_arm_force_controlled/meshes/geometry/connecting.stl" />
+    <xacro:property name="mesh_file_hebi" value="package://mav_arm_force_controlled/meshes/geometry/hebi.stl" />
+    <xacro:property name="mesh_file_hebitotube2" value="package://mav_arm_force_controlled/meshes/geometry/hebitotube2.stl" />
+    <xacro:property name="mesh_file_tube2" value="package://mav_arm_force_controlled/meshes/geometry/tube2.stl" />
+    <xacro:property name="mesh_file_clamp2" value="package://mav_arm_force_controlled/meshes/geometry/tube2todynamixel.stl" />
+    <xacro:property name="mesh_file_actuator1" value="package://mav_arm_force_controlled/meshes/geometry/dynamixel.stl" />
+    <xacro:property name="mesh_file_clamp1" value="package://mav_arm_force_controlled/meshes/geometry/dynamixeltotube1.stl" />
+    <xacro:property name="mesh_file_tube1" value="package://mav_arm_force_controlled/meshes/geometry/tube1.stl" />
+    <xacro:property name="mesh_file_tip" value="package://mav_arm_force_controlled/meshes/geometry/tip.stl" />
+    <!-- Mesh files of simplified geometry for collision checking-->
+    <xacro:property name="s_mesh_file_baseplate" value="package://mav_arm_force_controlled/meshes/simplified_geometry/baseplate.stl" />
+    <xacro:property name="s_mesh_file_dyamixel" value="package://mav_arm_force_controlled/meshes/simplified_geometry/dynamixel.stl" />
+    <xacro:property name="s_mesh_file_connecting" value="package://mav_arm_force_controlled/meshes/simplified_geometry/connecting.stl" />
+    <xacro:property name="s_mesh_file_hebi" value="package://mav_arm_force_controlled/meshes/simplified_geometry/hebi.stl" />
+    <xacro:property name="s_mesh_file_hebitotube2" value="package://mav_arm_force_controlled/meshes/simplified_geometry/hebitotube2.stl" />
+    <xacro:property name="s_mesh_file_tube2" value="package://mav_arm_force_controlled/meshes/simplified_geometry/tube2.stl" />
+    <xacro:property name="s_mesh_file_clamp2" value="package://mav_arm_force_controlled/meshes/simplified_geometry/tube2todynamixel.stl" />
+    <xacro:property name="s_mesh_file_actuator1" value="package://mav_arm_force_controlled/meshes/simplified_geometry/dynamixel.stl" />
+    <xacro:property name="s_mesh_file_clamp1" value="package://mav_arm_force_controlled/meshes/simplified_geometry/dynamixeltotube1.stl" />
+    <xacro:property name="s_mesh_file_tube1" value="package://mav_arm_force_controlled/meshes/simplified_geometry/tube1.stl" />
+    <xacro:property name="s_mesh_file_tip" value="package://mav_arm_force_controlled/meshes/simplified_geometry/tip.stl" />
     <!-- Mesh files are in mm. All mesh files are scaled by the factor 1000-->
     <xacro:property name="mesh_scale" value="0.001" />
@@ -64,5 +76,6 @@
     <collision>
       <geometry>
-        <box size="0.1 0.1 0.1"/>
+        <mesh filename="${s_mesh_file_baseplate}"
+              scale="${mesh_scale} ${mesh_scale} ${mesh_scale}"/>
         </geometry>
       <origin rpy="0 0 0" xyz="0 0 0"/>
@@ -99,5 +112,6 @@
     <collision>
       <geometry>
-        <box size="0.1 0.1 0.1"/>
+        <mesh filename="${s_mesh_file_dyamixel}"
+              scale="${mesh_scale} ${mesh_scale} ${mesh_scale}"/>
         </geometry>
       <origin rpy="0 0 0" xyz="0 0 0"/>
@@ -145,5 +159,6 @@
     <collision>
       <geometry>
-        <box size="0.1 0.1 0.1"/>
+        <mesh filename="${s_mesh_file_connecting}"
+              scale="${mesh_scale} ${mesh_scale} ${mesh_scale}"/>
         </geometry>
       <origin rpy="0 0 0" xyz="0 0 0"/>
@@ -180,5 +195,6 @@
     <collision>
       <geometry>
-        <box size="0.1 0.1 0.1"/>
+        <mesh filename="${s_mesh_file_hebi}"
+              scale="${mesh_scale} ${mesh_scale} ${mesh_scale}"/>
         </geometry>
       <origin rpy="0 0 0" xyz="0 0 0"/>
@@ -226,5 +242,6 @@
     <collision>
       <geometry>
-        <box size="0.1 0.1 0.1"/>
+        <mesh filename="${s_mesh_file_hebitotube2}"
+              scale="${mesh_scale} ${mesh_scale} ${mesh_scale}"/>
         </geometry>
       <origin rpy="0 0 0" xyz="0 0 0"/>
@@ -261,5 +278,6 @@
     <collision>
       <geometry>
-        <box size="0.1 0.1 0.1"/>
+        <mesh filename="${s_mesh_file_tube2}"
+              scale="${mesh_scale} ${mesh_scale} ${mesh_scale}"/>
         </geometry>
       <origin rpy="0 0 0" xyz="0 0 0"/>
@@ -296,5 +314,6 @@
       <collision>
         <geometry>
-          <box size="0.1 0.1 0.1"/>
+          <mesh filename="${s_mesh_file_clamp2}"
+                scale="${mesh_scale} ${mesh_scale} ${mesh_scale}"/>
           </geometry>
         <origin rpy="0 0 0" xyz="0 0 0"/>
@@ -331,5 +350,6 @@
       <collision>
         <geometry>
-          <box size="0.1 0.1 0.1"/>
+          <mesh filename="${s_mesh_file_actuator1}"
+            scale="${mesh_scale} ${mesh_scale} ${mesh_scale}"/>
           </geometry>
         <origin rpy="0 0 0" xyz="0 0 0"/>
@@ -377,5 +397,6 @@
     <collision>
       <geometry>
-        <box size="0.1 0.1 0.1"/>
+        <mesh filename="${s_mesh_file_clamp1}"
+          scale="${mesh_scale} ${mesh_scale} ${mesh_scale}"/>
         </geometry>
       <origin rpy="0 0 0" xyz="0 0 0"/>
@@ -412,5 +433,6 @@
       <collision>
         <geometry>
-          <box size="0.1 0.1 0.1"/>
+          <mesh filename="${s_mesh_file_tube1}"
+            scale="${mesh_scale} ${mesh_scale} ${mesh_scale}"/>
           </geometry>
         <origin rpy="0 0 0" xyz="0 0 0"/>
@@ -447,5 +469,6 @@
       <collision>
         <geometry>
-          <box size="0.1 0.1 0.1"/>
+          <mesh filename="${s_mesh_file_tip}"
+            scale="${mesh_scale} ${mesh_scale} ${mesh_scale}"/>
           </geometry>
         <origin rpy="0 0 0" xyz="0 0 0"/>
