Commit message: added more parts to the new arm form

File: src/fourth_model.urdf.xacro (robot description, xacro)
@@ -26,25 +26,42 @@
     <xacro:property name="mesh_file_baseplate" value="package://mav_arm_force_controlled/meshes/geometry_2.0/voliro_arm_base_dynamixel_balanced.stl" />
     <xacro:property name="mesh_file_dyamixel" value="package://mav_arm_force_controlled/meshes/geometry_2.0/voliro_arm_dynamixel.stl" />
+    <xacro:property name="mesh_file_dyamixel_to_hebi" value="package://mav_arm_force_controlled/meshes/geometry_2.0/voliro_arm_dynamixel_to_hebi.stl" />
+    <xacro:property name="mesh_file_hebi" value="package://mav_arm_force_controlled/meshes/geometry_2.0/voliro_arm_hebi.stl" />
+    <xacro:property name="mesh_file_clamp2" value="package://mav_arm_force_controlled/meshes/geometry_2.0/voliro_arm_clamp2.stl" />
+    <xacro:property name="mesh_file_tube2" value="package://mav_arm_force_controlled/meshes/geometry_2.0/voliro_arm_tube2.stl" />
+    <xacro:property name="mesh_file_tube_adapter" value="package://mav_arm_force_controlled/meshes/geometry_2.0/voliro_arm_tube_adapter.stl" />
+    <xacro:property name="mesh_file_actuator1" value="package://mav_arm_force_controlled/meshes/geometry_2.0/voliro_arm_dynamixel.stl" />
+    <xacro:property name="mesh_file_tube1" value="package://mav_arm_force_controlled/meshes/geometry_2.0/voliro_arm_tube1.stl" />
+    <xacro:property name="mesh_file_tip" value="package://mav_arm_force_controlled/meshes/geometry_2.0/voliro_arm_tip.stl" />
     <!-- Mesh files of simplified geometry for collision checking-->
     <xacro:property name="s_mesh_file_baseplate" value="package://mav_arm_force_controlled/meshes/simplified_geometry_2.0/voliro_arm_base_dynamixel_balanced.stl" />
     <xacro:property name="s_mesh_file_dyamixel" value="package://mav_arm_force_controlled/meshes/simplified_geometry_2.0/voliro_arm_dynamixel.stl" />
+    <xacro:property name="s_mesh_file_dyamixel_to_hebi" value="package://mav_arm_force_controlled/meshes/simplified_geometry_2.0/voliro_arm_dynamixel_to_hebi.stl" />
+    <xacro:property name="s_mesh_file_hebi" value="package://mav_arm_force_controlled/meshes/simplified_geometry_2.0/voliro_arm_hebi.stl" />
+    <xacro:property name="s_mesh_file_clamp2" value="package://mav_arm_force_controlled/meshes/simplified_geometry_2.0/voliro_arm_clamp2.stl" />
+    <xacro:property name="s_mesh_file_tube2" value="package://mav_arm_force_controlled/meshes/simplified_geometry_2.0/voliro_arm_tube2.stl" />
+    <xacro:property name="s_mesh_file_tube_adapter" value="package://mav_arm_force_controlled/meshes/simplified_geometry_2.0/voliro_arm_tube_adapter.stl" />
+    <xacro:property name="s_mesh_file_actuator1" value="package://mav_arm_force_controlled/meshes/simplified_geometry_2.0/voliro_arm_dynamixel.stl" />
+    <xacro:property name="s_mesh_file_tube1" value="package://mav_arm_force_controlled/meshes/simplified_geometry_2.0/voliro_arm_tube1.stl" />
+    <xacro:property name="s_mesh_file_tip" value="package://mav_arm_force_controlled/meshes/simplified_geometry_2.0/voliro_arm_tip.stl" />
     <!-- Mesh files are in mm. All mesh files are scaled by the factor 1000-->
     <xacro:property name="mesh_scale" value="0.001" />
     <!-- The Mass and inertia elements are defined before the link element-->
-    <xacro:property name="baseplate_mass" value="1" />
-    <xacro:property name="baseplate_cog_x" value="0.025202079" />
-    <xacro:property name="baseplate_cog_y" value="0" />
-    <xacro:property name="baseplate_cog_z" value="0.0025" />
-    <xacro:property name="baseplate_ixx" value="0.000063973" />
-    <xacro:property name="baseplate_ixy" value="0" />
-    <xacro:property name="baseplate_ixz" value="0.000005877" />
-    <xacro:property name="baseplate_iyy" value="0.000151767" />
-    <xacro:property name="baseplate_iyz" value="0" />
-    <xacro:property name="baseplate_izz" value="0.000214186" />
+    <xacro:property name="baseplate_mass" value="0.034534697" />
+    <xacro:property name="baseplate_cog_x" value="-0.0155840153" />
+    <xacro:property name="baseplate_cog_y" value="0.03245573125" />
+    <xacro:property name="baseplate_cog_z" value="0.01488134446" />
+<!-- To Do change units -->
+    <xacro:property name="baseplate_ixx" value="60.4589042" />
+    <xacro:property name="baseplate_ixy" value="-23.91373491" />
+    <xacro:property name="baseplate_ixz" value="-9.415308277" />
+    <xacro:property name="baseplate_iyy" value="32.25701807" />
+    <xacro:property name="baseplate_iyz" value="17.84460765" />
+    <xacro:property name="baseplate_izz" value="75.37700913" />
   <link name="world"/>
   <joint name="fixed" type="fixed">
     <parent link="world"/>
     <child link="baseplate"/>
-    <origin xyz="0.1 0.1 0" rpy="${pi} 0 0" />
+    <origin xyz="0.03244 0.0481 0.02" rpy="${pi} 0 0" />
   </joint>
   <link name="baseplate">
@@ -72,9 +89,9 @@
     <parent link="baseplate"/>
     <child link="actuator3"/>
-    <origin rpy="${pi} 0 ${pi}" xyz="0.1 0.1 0"/>
+    <origin rpy="${pi} 0 ${pi}" xyz="0 ${0.0425+0.0056} -0.017"/>
   </joint>
   <xacro:property name="dynamixel_mass" value="0.135" />
   <xacro:property name="dynamixel_cog_x" value="0.000000008" />
-  <xacro:property name="dynamixel_cog_y" value="-0.01519089" />
+  <xacro:property name="dynamixel_cog_y" value="0.01519089" />
   <xacro:property name="dynamixel_cog_z" value="0.000362847" />
   <xacro:property name="dynamixel_ixx" value="0.000129338" />
@@ -105,10 +122,9 @@
     </inertial>
   </link>
-<!--
-  <joint name="actuator_to_connectingbox" type="continuous">
-    <axis rpy="0 0 0" xyz="0 0 1"/>
+  <joint name="actuator_to_hebi" type="continuous">
+    <axis xyz="0 0 ${1}"/>
     <parent link="actuator3"/>
-    <child link="connectingbox"/>
-    <origin rpy="0 0 ${pi}" xyz="0 0 ${0.0235+0.0035}"/>
+    <child link="dynamixel_to_hebi"/>
+    <origin rpy="0 0 0" xyz="0 0 ${0.0235+0.012}"/>
     <limit effort="30" velocity="1.0"/>
   </joint>
@@ -118,22 +134,23 @@
       <mechanicalReduction>1</mechanicalReduction>
     </actuator>
-    <joint name="actuator_to_connectingbox">
+    <joint name="actuator_to_hebi">
       <hardwareInterface>hardware_interface/EffortJointInterface</hardwareInterface>
     </joint>
   </transmission>
-  <xacro:property name="connectionmx64hebi_mass" value=" 0.402140403" />
-  <xacro:property name="connectionmx64hebi_cog_x" value="0.000000171" />
-  <xacro:property name="connectionmx64hebi_cog_y" value="0.000278026" />
-  <xacro:property name="connectionmx64hebi_cog_z" value="0.038471524" />
-  <xacro:property name="connectionmx64hebi_ixx" value="0.001105121" />
-  <xacro:property name="connectionmx64hebi_ixy" value="0.000000016" />
-  <xacro:property name="connectionmx64hebi_ixz" value="0" />
-  <xacro:property name="connectionmx64hebi_iyy" value="0.001002814" />
-  <xacro:property name="connectionmx64hebi_iyz" value="0.000007088" />
-  <xacro:property name="connectionmx64hebi_izz" value="0.000170487" />
-  <link name="connectingbox">
-    <visual>
-      <geometry>
-        <mesh filename="${mesh_file_connecting}"
+<!-- To Do change unit -->
+  <xacro:property name="bearing_mass" value="0.123" />
+  <xacro:property name="bearing_cog_x" value="0.008737243596" />
+  <xacro:property name="bearing_cog_y" value="0.00095854858" />
+  <xacro:property name="bearing_cog_z" value="-0.01965454186" />
+  <xacro:property name="bearing_ixx" value="139.5553029" />
+  <xacro:property name="bearing_ixy" value="0.414376963" />
+  <xacro:property name="bearing_ixz" value="-31.92210758" />
+  <xacro:property name="bearing_iyy" value="162.416508" />
+  <xacro:property name="bearing_iyz" value="-0.344517543" />
+  <xacro:property name="bearing_izz" value="80.76641832" />
+  <link name="dynamixel_to_hebi">
+    <visual>
+      <geometry>
+        <mesh filename="${mesh_file_dyamixel_to_hebi}"
               scale="${mesh_scale} ${mesh_scale} ${mesh_scale}"/>
       </geometry>
@@ -143,18 +160,18 @@
     <collision>
       <geometry>
-        <mesh filename="${s_mesh_file_connecting}"
-              scale="${mesh_scale} ${mesh_scale} ${mesh_scale}"/>
-        </geometry>
-      <origin rpy="0 0 0" xyz="0 0 0"/>
-    </collision>
-    <inertial>
-      <mass value="${connectionmx64hebi_mass}"/>
-      <inertia ixx="${connectionmx64hebi_ixx}" ixy="${connectionmx64hebi_ixy}" ixz="${connectionmx64hebi_ixz}" iyy="${connectionmx64hebi_iyy}" iyz="${connectionmx64hebi_iyz}" izz="${connectionmx64hebi_izz}" />
+        <mesh filename="${s_mesh_file_dyamixel_to_hebi}"
+              scale="${mesh_scale} ${mesh_scale} ${mesh_scale}"/>
+        </geometry>
+      <origin rpy="0 0 0" xyz="0 0 0"/>
+    </collision>
+    <inertial>
+      <mass value="${bearing_mass}"/>
+      <inertia ixx="${bearing_ixx}" ixy="${bearing_ixy}" ixz="${bearing_ixz}" iyy="${bearing_iyy}" iyz="${bearing_iyz}" izz="${bearing_izz}" />
     </inertial>
   </link>
   <joint name="connectingbox_to_actuator2" type="fixed">
-    <parent link="connectingbox"/>
+    <parent link="dynamixel_to_hebi"/>
     <child link="actuator2"/>
-    <origin rpy="${pi/2} ${0} ${pi/2}"  xyz="${0.005+0.015} ${0} ${0.0635}"/>
+    <origin rpy="${pi/2} ${0} ${pi/2}"  xyz="${0.038+0.015} ${0} ${-0.029}"/>
   </joint>
   <xacro:property name="actuator2_mass" value="0.34" />
@@ -189,9 +206,10 @@
     </inertial>
   </link>
-  <joint name="actuator2_to_clamp3" type="continuous">
+  <joint name="actuator2_to_clamp2" type="continuous">
     <axis rpy="0 0 0" xyz="0 1 0"/>
     <parent link="actuator2"/>
-    <child link="clamp3"/>
-    <origin rpy="${pi/2} 0 ${-pi/2}" xyz="${0} 0 ${0.01605}"/>
+    <child link="clamp2"/>
+    <!--<origin rpy="${pi/2} ${0} ${-pi/2+pi/6}" xyz="${0} ${0} ${0.016}"/>-->
+    <origin rpy="${pi/2} ${0} ${-pi/2}" xyz="${0} ${0} ${0.01605}"/>
     <limit effort="30" velocity="1.0"/>
   </joint>
@@ -201,22 +219,23 @@
       <mechanicalReduction>1</mechanicalReduction>
     </actuator>
-    <joint name="actuator2_to_clamp3">
+    <joint name="actuator2_to_clamp2">
       <hardwareInterface>hardware_interface/EffortJointInterface</hardwareInterface>
     </joint>
   </transmission>
-  <xacro:property name="clamp3_mass" value="0.21" />
-  <xacro:property name="clamp3_cog_x" value="0.015022968" />
-  <xacro:property name="clamp3_cog_y" value="0.001776283" />
-  <xacro:property name="clamp3_cog_z" value="0.000017898" />
-  <xacro:property name="clamp3_ixx" value="0.000524947" />
-  <xacro:property name="clamp3_ixy" value="0.000000017" />
-  <xacro:property name="clamp3_ixz" value="-0.00000004" />
-  <xacro:property name="clamp3_iyy" value="0.000535726" />
-  <xacro:property name="clamp3_iyz" value="-0.000092479" />
-  <xacro:property name="clamp3_izz" value="0.000074342" />
-  <link name="clamp3">
-    <visual>
-      <geometry>
-        <mesh filename="${mesh_file_hebitotube2}"
+  <xacro:property name="clamp2_mass" value="0.029" />
+  <xacro:property name="clamp2_cog_x" value="0.00000000019" />
+  <xacro:property name="clamp2_cog_y" value="0.008.118243555" />
+  <xacro:property name="clamp2_cog_z" value="-0.01350332735" />
+<!-- To do change units-->
+  <xacro:property name="clamp2_ixx" value="21.61924342" />
+  <xacro:property name="clamp2_ixy" value="-0.000002107" />
+  <xacro:property name="clamp2_ixz" value="0.000000228" />
+  <xacro:property name="clamp2_iyy" value="23.46303475" />
+  <xacro:property name="clamp2_iyz" value="-4.826007788" />
+  <xacro:property name="clamp2_izz" value="7.990509672" />
+  <link name="clamp2">
+    <visual>
+      <geometry>
+        <mesh filename="${mesh_file_clamp2}"
               scale="${mesh_scale} ${mesh_scale} ${mesh_scale}"/>
       </geometry>
@@ -226,18 +245,18 @@
     <collision>
       <geometry>
-        <mesh filename="${s_mesh_file_hebitotube2}"
-              scale="${mesh_scale} ${mesh_scale} ${mesh_scale}"/>
-        </geometry>
-      <origin rpy="0 0 0" xyz="0 0 0"/>
-    </collision>
-    <inertial>
-      <mass value="${clamp3_mass}"/>
-      <inertia ixx="${clamp3_ixx}" ixy="${clamp3_ixy}" ixz="${clamp3_ixz}" iyy="${clamp3_iyy}" iyz="${clamp3_iyz}" izz="${clamp3_izz}" />
-    </inertial>
-  </link>
-  <joint name="clamp3_to_tube2" type="fixed">
-    <parent link="clamp3"/>
+        <mesh filename="${s_mesh_file_clamp2}"
+              scale="${mesh_scale} ${mesh_scale} ${mesh_scale}"/>
+        </geometry>
+      <origin rpy="0 0 0" xyz="0 0 0"/>
+    </collision>
+    <inertial>
+      <mass value="${clamp2_mass}"/>
+      <inertia ixx="${clamp2_ixx}" ixy="${clamp2_ixy}" ixz="${clamp2_ixz}" iyy="${clamp2_iyy}" iyz="${clamp2_iyz}" izz="${clamp2_izz}" />
+    </inertial>
+  </link>
+  <joint name="clamp2_to_tube2" type="fixed">
+    <parent link="clamp2"/>
     <child link="tube2"/>
-    <origin rpy="0 ${pi} 0" xyz="${0} ${0.013} ${-0.035}"/>
+    <origin rpy="0 ${pi} 0" xyz="${0} ${0.012} ${-0.02}"/>
   </joint>
   <xacro:property name="tube2_mass" value="0.038201767" />
@@ -274,21 +293,22 @@
     <joint name="tube2_to_clamp2" type="fixed">
       <parent link="tube2"/>
-      <child link="clamp2"/>
-      <origin rpy="${pi/2} 0 ${-pi}" xyz="${0} ${-0.018} ${0.4-0.055}"/>
+      <child link="tube_adapter"/>
+      <origin rpy="${pi/2} 0 ${-pi}" xyz="${0} ${-0.02} ${0.4-0.0056}"/>
     </joint>
-    <xacro:property name="clamp2_mass" value="0.128888247" />
-    <xacro:property name="clamp2_cog_x" value="0.000000004" />
-    <xacro:property name="clamp2_cog_y" value="0.02936423" />
-    <xacro:property name="clamp2_cog_z" value="0.016233149" />
-    <xacro:property name="clamp2_ixx" value="0.00019462" />
-    <xacro:property name="clamp2_ixy" value="0" />
-    <xacro:property name="clamp2_ixz" value="0" />
-    <xacro:property name="clamp2_iyy" value="0.000067787" />
-    <xacro:property name="clamp2_iyz" value="0.000060459" />
-    <xacro:property name="clamp2_izz" value="0.000173715" />
-    <link name="clamp2">
+    <xacro:property name="clamp2_mass" value="0.027727776" />
+    <xacro:property name="clamp2_cog_x" value="-0.000051031" />
+    <xacro:property name="clamp2_cog_y" value="-5.987489264" />
+    <xacro:property name="clamp2_cog_z" value="20" />
+    <!-- To Do change units -->
+    <xacro:property name="clamp2_ixx" value="27.76777587" />
+    <xacro:property name="clamp2_ixy" value="0.000019714" />
+    <xacro:property name="clamp2_ixz" value="-0.00001739" />
+    <xacro:property name="clamp2_iyy" value="21.78807802" />
+    <xacro:property name="clamp2_iyz" value="-3.320450023" />
+    <xacro:property name="clamp2_izz" value="14.62444632" />
+    <link name="tube_adapter">
       <visual>
         <geometry>
-          <mesh filename="${mesh_file_clamp2}"
+          <mesh filename="${mesh_file_tube_adapter}"
                 scale="${mesh_scale} ${mesh_scale} ${mesh_scale}"/>
         </geometry>
@@ -298,5 +318,5 @@
       <collision>
         <geometry>
-          <mesh filename="${s_mesh_file_clamp2}"
+          <mesh filename="${s_mesh_file_tube_adapter}"
                 scale="${mesh_scale} ${mesh_scale} ${mesh_scale}"/>
           </geometry>
@@ -309,9 +329,9 @@
     </link>
       <joint name="clamp2_to_actuator1" type="fixed">
-        <parent link="clamp2"/>
+        <parent link="tube_adapter"/>
         <child link="actuator1"/>
-        <origin rpy="0 ${pi} 0" xyz="${0} ${0.0056+0.0425} ${-0.017}"/>
+        <origin rpy="0 ${pi} 0" xyz="${0} ${0.0425+0.0056} ${0.017+0.003}"/>
       </joint>
-      <xacro:property name="actuator1_mass" value="0.126" />
+      <xacro:property name="actuator1_mass" value="0.135" />
       <xacro:property name="actuator1_cog_x" value="0.000000008" />
       <xacro:property name="actuator1_cog_y" value="-0.01519089" />
@@ -344,4 +364,5 @@
       </inertial>
     </link>
+  <!--
   <joint name="actuator1_to_clamp1" type="continuous">
     <axis rpy="0 0 0" xyz="0 0 1"/>

Commit message: finalized new arm form

File: src/fourth_model.urdf.xacro (robot description, xacro)
@@ -32,4 +32,5 @@
     <xacro:property name="mesh_file_tube_adapter" value="package://mav_arm_force_controlled/meshes/geometry_2.0/voliro_arm_tube_adapter.stl" />
     <xacro:property name="mesh_file_actuator1" value="package://mav_arm_force_controlled/meshes/geometry_2.0/voliro_arm_dynamixel.stl" />
+    <xacro:property name="mesh_file_clamp1" value="package://mav_arm_force_controlled/meshes/geometry_2.0/voliro_arm_clamp1.stl" />
     <xacro:property name="mesh_file_tube1" value="package://mav_arm_force_controlled/meshes/geometry_2.0/voliro_arm_tube1.stl" />
     <xacro:property name="mesh_file_tip" value="package://mav_arm_force_controlled/meshes/geometry_2.0/voliro_arm_tip.stl" />
@@ -43,4 +44,5 @@
     <xacro:property name="s_mesh_file_tube_adapter" value="package://mav_arm_force_controlled/meshes/simplified_geometry_2.0/voliro_arm_tube_adapter.stl" />
     <xacro:property name="s_mesh_file_actuator1" value="package://mav_arm_force_controlled/meshes/simplified_geometry_2.0/voliro_arm_dynamixel.stl" />
+    <xacro:property name="s_mesh_file_clamp1" value="package://mav_arm_force_controlled/meshes/simplified_geometry_2.0/voliro_arm_clamp1.stl" />
     <xacro:property name="s_mesh_file_tube1" value="package://mav_arm_force_controlled/meshes/simplified_geometry_2.0/voliro_arm_tube1.stl" />
     <xacro:property name="s_mesh_file_tip" value="package://mav_arm_force_controlled/meshes/simplified_geometry_2.0/voliro_arm_tip.stl" />
@@ -364,10 +366,9 @@
       </inertial>
     </link>
-  <!--
   <joint name="actuator1_to_clamp1" type="continuous">
     <axis rpy="0 0 0" xyz="0 0 1"/>
     <parent link="actuator1"/>
     <child link="clamp1"/>
-    <origin rpy="${0} ${0} ${-pi/2}" xyz="${0} ${0} ${0.0235}"/>
+    <origin rpy="${0} ${0} ${0}" xyz="${0} ${0} ${0.0235}"/>
     <limit effort="30" velocity="1.0"/>
   </joint>
@@ -381,14 +382,15 @@
     </joint>
   </transmission>
-  <xacro:property name="clamp1_mass" value="0.11739877" />
-  <xacro:property name="clamp1_cog_x" value="0.008717092" />
-  <xacro:property name="clamp1_cog_y" value="0.000001711" />
-  <xacro:property name="clamp1_cog_z" value="0.011234631" />
-  <xacro:property name="clamp1_ixx" value="0.000045773" />
-  <xacro:property name="clamp1_ixy" value="-0.00000003" />
-  <xacro:property name="clamp1_ixz" value="0.000022588" />
-  <xacro:property name="clamp1_iyy" value="0.000079456" />
-  <xacro:property name="clamp1_iyz" value="0.000000001" />
-  <xacro:property name="clamp1_izz" value="0.00007801" />
+  <xacro:property name="clamp1_mass" value="0.084238767" />
+  <xacro:property name="clamp1_cog_x" value="-0.000000709384" />
+  <xacro:property name="clamp1_cog_y" value="0.003831382911" />
+  <xacro:property name="clamp1_cog_z" value="0.007840028704" />
+ <!-- Todo change units -->
+  <xacro:property name="clamp1_ixx" value="35.98639204" />
+  <xacro:property name="clamp1_ixy" value="-0.036707373" />
+  <xacro:property name="clamp1_ixz" value="-0.00032096" />
+  <xacro:property name="clamp1_iyy" value="26.23411723" />
+  <xacro:property name="clamp1_iyz" value="7.078559572" />
+  <xacro:property name="clamp1_izz" value="43.83528986" />
   <link name="clamp1">
     <visual>
@@ -415,5 +417,5 @@
     <parent link="clamp1"/>
     <child link="tube1"/>
-    <origin rpy="${0} ${pi/2} ${0}" xyz="${0.015} ${0} ${0.022}"/>
+    <origin rpy="${0} ${pi/2} ${pi/2}" xyz="${0} ${0.016} ${0.022}"/>
   </joint>
   <xacro:property name="tube1_mass" value="0.02035752" />
@@ -453,14 +455,15 @@
       <origin rpy="${0} ${0} ${0}" xyz="${0} ${0} ${0.6}"/>
     </joint>
-    <xacro:property name="tip_mass" value="0.039351907" />
+    <xacro:property name="tip_mass" value="0.001658447" />
     <xacro:property name="tip_cog_x" value="0" />
     <xacro:property name="tip_cog_y" value="0" />
     <xacro:property name="tip_cog_z" value="0.000163952" />
-    <xacro:property name="tip_ixx" value="0.000000758" />
+<!-- To Do change units -->
+    <xacro:property name="tip_ixx" value="0.031944763" />
     <xacro:property name="tip_ixy" value="0" />
     <xacro:property name="tip_ixz" value="0" />
-    <xacro:property name="tip_iyy" value="0.000000758" />
+    <xacro:property name="tip_iyy" value="0.031944763" />
     <xacro:property name="tip_iyz" value="0" />
-    <xacro:property name="tip_izz" value="0.0000008" />
+    <xacro:property name="tip_izz" value="0.033720057" />
     <link name="tip">
       <visual>
@@ -484,5 +487,4 @@
       </inertial>
     </link>
--->
     <gazebo>
       <plugin name="gazebo_ros_control" filename="libgazebo_ros_control.so">
