Commit message: corrected inertia units

File: src/fourth_model.urdf.xacro (robot description, xacro)
@@ -49,4 +49,6 @@
     <!-- Mesh files are in mm. All mesh files are scaled by the factor 1000-->
     <xacro:property name="mesh_scale" value="0.001" />
+    <!-- Unit conversion for inertia from kg*mm² to kg m² -->
+    <xacro:property name="uc_inertia" value="0.000001" />
     <!-- The Mass and inertia elements are defined before the link element-->
     <xacro:property name="baseplate_mass" value="0.034534697" />
@@ -55,10 +57,10 @@
     <xacro:property name="baseplate_cog_z" value="0.01488134446" />
 <!-- To Do change units -->
-    <xacro:property name="baseplate_ixx" value="60.4589042" />
-    <xacro:property name="baseplate_ixy" value="-23.91373491" />
-    <xacro:property name="baseplate_ixz" value="-9.415308277" />
-    <xacro:property name="baseplate_iyy" value="32.25701807" />
-    <xacro:property name="baseplate_iyz" value="17.84460765" />
-    <xacro:property name="baseplate_izz" value="75.37700913" />
+    <xacro:property name="baseplate_ixx" value="${60.4589042*uc_inertia}" />
+    <xacro:property name="baseplate_ixy" value="${-23.91373491*uc_inertia}" />
+    <xacro:property name="baseplate_ixz" value="${-9.415308277*uc_inertia}" />
+    <xacro:property name="baseplate_iyy" value="${32.25701807*uc_inertia}" />
+    <xacro:property name="baseplate_iyz" value="${17.84460765*uc_inertia}" />
+    <xacro:property name="baseplate_izz" value="${75.37700913*uc_inertia}" />
   <link name="world"/>
   <joint name="fixed" type="fixed">
@@ -145,10 +147,10 @@
   <xacro:property name="bearing_cog_y" value="0.00095854858" />
   <xacro:property name="bearing_cog_z" value="-0.01965454186" />
-  <xacro:property name="bearing_ixx" value="139.5553029" />
-  <xacro:property name="bearing_ixy" value="0.414376963" />
-  <xacro:property name="bearing_ixz" value="-31.92210758" />
-  <xacro:property name="bearing_iyy" value="162.416508" />
-  <xacro:property name="bearing_iyz" value="-0.344517543" />
-  <xacro:property name="bearing_izz" value="80.76641832" />
+  <xacro:property name="bearing_ixx" value="${139.5553029*uc_inertia}" />
+  <xacro:property name="bearing_ixy" value="${0.414376963*uc_inertia}" />
+  <xacro:property name="bearing_ixz" value="${-31.92210758*uc_inertia}" />
+  <xacro:property name="bearing_iyy" value="${162.416508*uc_inertia}" />
+  <xacro:property name="bearing_iyz" value="${-0.344517543*uc_inertia}" />
+  <xacro:property name="bearing_izz" value="${80.76641832*uc_inertia}" />
   <link name="dynamixel_to_hebi">
     <visual>
@@ -212,5 +214,4 @@
     <parent link="actuator2"/>
     <child link="clamp2"/>
-    <!--<origin rpy="${pi/2} ${0} ${-pi/2+pi/6}" xyz="${0} ${0} ${0.016}"/>-->
     <origin rpy="${pi/2} ${0} ${-pi/2}" xyz="${0} ${0} ${0.01605}"/>
     <limit effort="30" velocity="1.0"/>
@@ -230,10 +231,10 @@
   <xacro:property name="clamp2_cog_z" value="-0.01350332735" />
 <!-- To do change units-->
-  <xacro:property name="clamp2_ixx" value="21.61924342" />
-  <xacro:property name="clamp2_ixy" value="-0.000002107" />
-  <xacro:property name="clamp2_ixz" value="0.000000228" />
-  <xacro:property name="clamp2_iyy" value="23.46303475" />
-  <xacro:property name="clamp2_iyz" value="-4.826007788" />
-  <xacro:property name="clamp2_izz" value="7.990509672" />
+  <xacro:property name="clamp2_ixx" value="${21.61924342*uc_inertia}" />
+  <xacro:property name="clamp2_ixy" value="${-0.000002107*uc_inertia}" />
+  <xacro:property name="clamp2_ixz" value="${0.000000228*uc_inertia}" />
+  <xacro:property name="clamp2_iyy" value="${23.46303475*uc_inertia}" />
+  <xacro:property name="clamp2_iyz" value="${-4.826007788*uc_inertia}" />
+  <xacro:property name="clamp2_izz" value="${7.990509672*uc_inertia}" />
   <link name="clamp2">
     <visual>
@@ -293,5 +294,5 @@
     </inertial>
   </link>
-    <joint name="tube2_to_clamp2" type="fixed">
+    <joint name="tube2_to_adapter" type="fixed">
       <parent link="tube2"/>
       <child link="tube_adapter"/>
@@ -303,10 +304,10 @@
     <xacro:property name="clamp2_cog_z" value="20" />
     <!-- To Do change units -->
-    <xacro:property name="clamp2_ixx" value="27.76777587" />
-    <xacro:property name="clamp2_ixy" value="0.000019714" />
-    <xacro:property name="clamp2_ixz" value="-0.00001739" />
-    <xacro:property name="clamp2_iyy" value="21.78807802" />
-    <xacro:property name="clamp2_iyz" value="-3.320450023" />
-    <xacro:property name="clamp2_izz" value="14.62444632" />
+    <xacro:property name="clamp2_ixx" value="${27.76777587*uc_inertia}" />
+    <xacro:property name="clamp2_ixy" value="${0.000019714*uc_inertia}" />
+    <xacro:property name="clamp2_ixz" value="${-0.00001739*uc_inertia}" />
+    <xacro:property name="clamp2_iyy" value="${21.78807802*uc_inertia}" />
+    <xacro:property name="clamp2_iyz" value="${-3.320450023*uc_inertia}" />
+    <xacro:property name="clamp2_izz" value="${14.62444632*uc_inertia}" />
     <link name="tube_adapter">
       <visual>
@@ -387,10 +388,10 @@
   <xacro:property name="clamp1_cog_z" value="0.007840028704" />
  <!-- Todo change units -->
-  <xacro:property name="clamp1_ixx" value="35.98639204" />
-  <xacro:property name="clamp1_ixy" value="-0.036707373" />
-  <xacro:property name="clamp1_ixz" value="-0.00032096" />
-  <xacro:property name="clamp1_iyy" value="26.23411723" />
-  <xacro:property name="clamp1_iyz" value="7.078559572" />
-  <xacro:property name="clamp1_izz" value="43.83528986" />
+  <xacro:property name="clamp1_ixx" value="${35.98639204*uc_inertia}" />
+  <xacro:property name="clamp1_ixy" value="${-0.036707373*uc_inertia}" />
+  <xacro:property name="clamp1_ixz" value="${-0.00032096*uc_inertia}" />
+  <xacro:property name="clamp1_iyy" value="${26.23411723*uc_inertia}" />
+  <xacro:property name="clamp1_iyz" value="${7.078559572*uc_inertia}" />
+  <xacro:property name="clamp1_izz" value="${43.83528986*uc_inertia}" />
   <link name="clamp1">
     <visual>
@@ -460,10 +461,10 @@
     <xacro:property name="tip_cog_z" value="0.000163952" />
 <!-- To Do change units -->
-    <xacro:property name="tip_ixx" value="0.031944763" />
-    <xacro:property name="tip_ixy" value="0" />
-    <xacro:property name="tip_ixz" value="0" />
-    <xacro:property name="tip_iyy" value="0.031944763" />
-    <xacro:property name="tip_iyz" value="0" />
-    <xacro:property name="tip_izz" value="0.033720057" />
+    <xacro:property name="tip_ixx" value="${0.031944763*uc_inertia}" />
+    <xacro:property name="tip_ixy" value="${0*uc_inertia}" />
+    <xacro:property name="tip_ixz" value="${0*uc_inertia}" />
+    <xacro:property name="tip_iyy" value="${0.031944763*uc_inertia}" />
+    <xacro:property name="tip_iyz" value="${0*uc_inertia}" />
+    <xacro:property name="tip_izz" value="${0.033720057*uc_inertia}" />
     <link name="tip">
       <visual>
@@ -498,5 +499,5 @@
       <selfCollide>true</selfCollide>
     </gazebo>
-    <gazebo reference="connectingbox">
+    <gazebo reference="dynamixel_to_hebi">
       <selfCollide>true</selfCollide>
     </gazebo>
@@ -504,5 +505,5 @@
       <selfCollide>true</selfCollide>
     </gazebo>
-    <gazebo reference="clamp3">
+    <gazebo reference="clamp2">
       <selfCollide>true</selfCollide>
     </gazebo>
@@ -510,5 +511,5 @@
       <selfCollide>true</selfCollide>
     </gazebo>
-    <gazebo reference="clamp2">
+    <gazebo reference="tube_adapter">
       <selfCollide>true</selfCollide>
     </gazebo>

Commit message: corrected clamp2 collision file

File: src/fourth_model.urdf.xacro (robot description, xacro)
@@ -56,5 +56,4 @@
     <xacro:property name="baseplate_cog_y" value="0.03245573125" />
     <xacro:property name="baseplate_cog_z" value="0.01488134446" />
-<!-- To Do change units -->
     <xacro:property name="baseplate_ixx" value="${60.4589042*uc_inertia}" />
     <xacro:property name="baseplate_ixy" value="${-23.91373491*uc_inertia}" />
@@ -142,5 +141,4 @@
     </joint>
   </transmission>
-<!-- To Do change unit -->
   <xacro:property name="bearing_mass" value="0.123" />
   <xacro:property name="bearing_cog_x" value="0.008737243596" />
@@ -215,5 +213,5 @@
     <child link="clamp2"/>
     <origin rpy="${pi/2} ${0} ${-pi/2}" xyz="${0} ${0} ${0.01605}"/>
-    <limit effort="30" velocity="1.0"/>
+    <limit effort="100" velocity="1.0"/>
   </joint>
   <transmission name="actuator2_hebi_trans">
@@ -230,5 +228,4 @@
   <xacro:property name="clamp2_cog_y" value="0.008.118243555" />
   <xacro:property name="clamp2_cog_z" value="-0.01350332735" />
-<!-- To do change units-->
   <xacro:property name="clamp2_ixx" value="${21.61924342*uc_inertia}" />
   <xacro:property name="clamp2_ixy" value="${-0.000002107*uc_inertia}" />
@@ -303,5 +300,4 @@
     <xacro:property name="clamp2_cog_y" value="-5.987489264" />
     <xacro:property name="clamp2_cog_z" value="20" />
-    <!-- To Do change units -->
     <xacro:property name="clamp2_ixx" value="${27.76777587*uc_inertia}" />
     <xacro:property name="clamp2_ixy" value="${0.000019714*uc_inertia}" />
@@ -372,5 +368,5 @@
     <child link="clamp1"/>
     <origin rpy="${0} ${0} ${0}" xyz="${0} ${0} ${0.0235}"/>
-    <limit effort="30" velocity="1.0"/>
+    <limit effort="100" velocity="1.0"/>
   </joint>
   <transmission name="actuator1_dynamixel_trans">
@@ -387,5 +383,4 @@
   <xacro:property name="clamp1_cog_y" value="0.003831382911" />
   <xacro:property name="clamp1_cog_z" value="0.007840028704" />
- <!-- Todo change units -->
   <xacro:property name="clamp1_ixx" value="${35.98639204*uc_inertia}" />
   <xacro:property name="clamp1_ixy" value="${-0.036707373*uc_inertia}" />
@@ -460,5 +455,4 @@
     <xacro:property name="tip_cog_y" value="0" />
     <xacro:property name="tip_cog_z" value="0.000163952" />
-<!-- To Do change units -->
     <xacro:property name="tip_ixx" value="${0.031944763*uc_inertia}" />
     <xacro:property name="tip_ixy" value="${0*uc_inertia}" />

Commit message: changed joint type from continious --> jittered to revolute --> stable

File: src/fourth_model.urdf.xacro (robot description, xacro)
@@ -125,9 +125,9 @@
     </inertial>
   </link>
-  <joint name="actuator_to_hebi" type="continuous">
-    <axis xyz="0 0 ${1}"/>
+  <joint name="actuator_to_hebi" type="revolute">
+    <axis rpy="0 0 0" xyz="0 0 1"/>
     <parent link="actuator3"/>
     <child link="dynamixel_to_hebi"/>
-    <origin rpy="0 0 0" xyz="0 0 ${0.0235+0.012}"/>
+    <origin rpy="0 0 ${0}" xyz="0 0 ${0.0235+0.012}"/>
     <limit effort="30" velocity="1.0"/>
   </joint>
@@ -172,5 +172,5 @@
     </inertial>
   </link>
-  <joint name="connectingbox_to_actuator2" type="fixed">
+  <joint name="bearing_to_actuator2" type="fixed">
     <parent link="dynamixel_to_hebi"/>
     <child link="actuator2"/>
@@ -208,10 +208,10 @@
     </inertial>
   </link>
-  <joint name="actuator2_to_clamp2" type="continuous">
+  <joint name="actuator2_to_clamp2" type="revolute">
     <axis rpy="0 0 0" xyz="0 1 0"/>
     <parent link="actuator2"/>
     <child link="clamp2"/>
-    <origin rpy="${pi/2} ${0} ${-pi/2}" xyz="${0} ${0} ${0.01605}"/>
-    <limit effort="100" velocity="1.0"/>
+    <origin rpy="${pi/2} ${0} ${0}" xyz="${0} ${0} ${0.01605}"/>
+    <limit effort="30" velocity="1.0"/>
   </joint>
   <transmission name="actuator2_hebi_trans">
@@ -296,14 +296,14 @@
       <origin rpy="${pi/2} 0 ${-pi}" xyz="${0} ${-0.02} ${0.4-0.0056}"/>
     </joint>
-    <xacro:property name="clamp2_mass" value="0.027727776" />
+    <xacro:property name="clamp2_mass" value="0.02919169" />
     <xacro:property name="clamp2_cog_x" value="-0.000051031" />
     <xacro:property name="clamp2_cog_y" value="-5.987489264" />
     <xacro:property name="clamp2_cog_z" value="20" />
-    <xacro:property name="clamp2_ixx" value="${27.76777587*uc_inertia}" />
-    <xacro:property name="clamp2_ixy" value="${0.000019714*uc_inertia}" />
-    <xacro:property name="clamp2_ixz" value="${-0.00001739*uc_inertia}" />
-    <xacro:property name="clamp2_iyy" value="${21.78807802*uc_inertia}" />
-    <xacro:property name="clamp2_iyz" value="${-3.320450023*uc_inertia}" />
-    <xacro:property name="clamp2_izz" value="${14.62444632*uc_inertia}" />
+    <xacro:property name="clamp2_ixx" value="${21.61924342*uc_inertia}" />
+    <xacro:property name="clamp2_ixy" value="${-0.000002107*uc_inertia}" />
+    <xacro:property name="clamp2_ixz" value="${0.000000228*uc_inertia}" />
+    <xacro:property name="clamp2_iyy" value="${23.46303475*uc_inertia}" />
+    <xacro:property name="clamp2_iyz" value="${-4.826007788*uc_inertia}" />
+    <xacro:property name="clamp2_izz" value="${7.990509672*uc_inertia}" />
     <link name="tube_adapter">
       <visual>
@@ -363,10 +363,10 @@
       </inertial>
     </link>
-  <joint name="actuator1_to_clamp1" type="continuous">
+  <joint name="actuator1_to_clamp1" type="revolute">
     <axis rpy="0 0 0" xyz="0 0 1"/>
     <parent link="actuator1"/>
     <child link="clamp1"/>
     <origin rpy="${0} ${0} ${0}" xyz="${0} ${0} ${0.0235}"/>
-    <limit effort="100" velocity="1.0"/>
+    <limit effort="30" velocity="1.0"/>
   </joint>
   <transmission name="actuator1_dynamixel_trans">
@@ -482,4 +482,5 @@
       </inertial>
     </link>
+revolute
     <gazebo>
       <plugin name="gazebo_ros_control" filename="libgazebo_ros_control.so">

File: src/thirdmodel.urdf.xacro (robot description, xacro)
@@ -123,5 +123,5 @@
     </inertial>
   </link>
-  <joint name="actuator_to_connectingbox" type="continuous">
+  <joint name="actuator_to_connectingbox" type="revolute">
     <axis rpy="0 0 0" xyz="0 0 1"/>
     <parent link="actuator3"/>
@@ -206,5 +206,5 @@
     </inertial>
   </link>
-  <joint name="actuator2_to_clamp3" type="continuous">
+  <joint name="actuator2_to_clamp3" type="revolute">
     <axis rpy="0 0 0" xyz="0 1 0"/>
     <parent link="actuator2"/>
@@ -361,5 +361,5 @@
       </inertial>
     </link>
-  <joint name="actuator1_to_clamp1" type="continuous">
+  <joint name="actuator1_to_clamp1" type="revolute">
     <axis rpy="0 0 0" xyz="0 0 1"/>
     <parent link="actuator1"/>

Commit message: changed joint type, stable gazebo, changed PID values

File: src/fourth_model.urdf.xacro (robot description, xacro)
@@ -22,5 +22,5 @@
   </material>
     <!-- General Variables-->
-    <xacro:property name="pi" value="3.1415269" />
+    <xacro:property name="pi" value="3.1415926535897931" />
     <!-- Mesh files of exact geometry-->
     <xacro:property name="mesh_file_baseplate" value="package://mav_arm_force_controlled/meshes/geometry_2.0/voliro_arm_base_dynamixel_balanced.stl" />
@@ -114,5 +114,5 @@
     </visual>
     <collision>
-      <geometry>
+      <geometry>s
         <mesh filename="${s_mesh_file_dyamixel}"
               scale="${mesh_scale} ${mesh_scale} ${mesh_scale}"/>
@@ -129,15 +129,17 @@
     <parent link="actuator3"/>
     <child link="dynamixel_to_hebi"/>
-    <origin rpy="0 0 ${0}" xyz="0 0 ${0.0235+0.012}"/>
-    <limit effort="30" velocity="1.0"/>
+    <origin rpy="0 0 ${pi/2}" xyz="0 0 ${0.0235+0.012}"/>
+    <!--<limit effort="100" velocity="10"/>-->
+    <limit effort="100" lower="${-pi/2}" upper="${pi/2}" velocity="10" />
   </joint>
   <transmission name="actuator3_dynamixel_trans">
     <type>transmission_interface/SimpleTransmission</type>
-    <actuator name="actuator3_dynamixel_motor">
-      <mechanicalReduction>1</mechanicalReduction>
-    </actuator>
     <joint name="actuator_to_hebi">
       <hardwareInterface>hardware_interface/EffortJointInterface</hardwareInterface>
     </joint>
+    <actuator name="actuator3_dynamixel_motor">
+      <hardwareInterface>hardware_interface/EffortJointInterface</hardwareInterface>
+      <mechanicalReduction>1</mechanicalReduction>
+    </actuator>
   </transmission>
   <xacro:property name="bearing_mass" value="0.123" />
@@ -208,10 +210,11 @@
     </inertial>
   </link>
-  <joint name="actuator2_to_clamp2" type="revolute">
-    <axis rpy="0 0 0" xyz="0 1 0"/>
+  <joint name="actuator2_to_clamp2" type="continuous">
+    <axis rpy="0 0 0" xyz="0 -1 0"/>
     <parent link="actuator2"/>
     <child link="clamp2"/>
     <origin rpy="${pi/2} ${0} ${0}" xyz="${0} ${0} ${0.01605}"/>
-    <limit effort="30" velocity="1.0"/>
+    <limit effort="100" velocity="10" />
+    <!--<limit effort="100" lower="${-2*pi}" upper="${2*pi}" velocity="10" />-->
   </joint>
   <transmission name="actuator2_hebi_trans">
@@ -363,19 +366,21 @@
       </inertial>
     </link>
-  <joint name="actuator1_to_clamp1" type="revolute">
+  <joint name="actuator1_to_clamp1" type="continuous">
     <axis rpy="0 0 0" xyz="0 0 1"/>
     <parent link="actuator1"/>
     <child link="clamp1"/>
     <origin rpy="${0} ${0} ${0}" xyz="${0} ${0} ${0.0235}"/>
-    <limit effort="30" velocity="1.0"/>
+    <limit effort="100" velocity="10" />
+    <!--<limit effort="100" lower="${-2*pi}" upper="${2*pi}" velocity="10" />-->
   </joint>
   <transmission name="actuator1_dynamixel_trans">
     <type>transmission_interface/SimpleTransmission</type>
-    <actuator name="$actuator1_dynamixel_motor">
-      <mechanicalReduction>1</mechanicalReduction>
-    </actuator>
     <joint name="actuator1_to_clamp1">
       <hardwareInterface>hardware_interface/EffortJointInterface</hardwareInterface>
     </joint>
+    <actuator name="actuator1_dynamixel">
+      <hardwareInterface>hardware_interface/EffortJointInterface</hardwareInterface>
+      <mechanicalReduction>1</mechanicalReduction>
+    </actuator>
   </transmission>
   <xacro:property name="clamp1_mass" value="0.084238767" />
@@ -482,8 +487,8 @@
       </inertial>
     </link>
-revolute
     <gazebo>
       <plugin name="gazebo_ros_control" filename="libgazebo_ros_control.so">
         <robotNamespace>/arm</robotNamespace>
+        <robotSimType>gazebo_ros_control/DefaultRobotHWSim</robotSimType>
       </plugin>
     </gazebo>
@@ -521,4 +526,3 @@
       <selfCollide>true</selfCollide>
     </gazebo>
-        <!--<robotSimType>gazebo_ros_control/DefaultRobotHWSim</robotSimType>-->
 </robot>

Commit message: added realistic limits

File: src/fourth_model.urdf.xacro (robot description, xacro)
@@ -131,5 +131,5 @@
     <origin rpy="0 0 ${pi/2}" xyz="0 0 ${0.0235+0.012}"/>
     <!--<limit effort="100" velocity="10"/>-->
-    <limit effort="100" lower="${-pi/2}" upper="${pi/2}" velocity="10" />
+    <limit effort="5" lower="${-pi/2}" upper="${pi/2}" velocity="1" />
   </joint>
   <transmission name="actuator3_dynamixel_trans">
@@ -215,5 +215,5 @@
     <child link="clamp2"/>
     <origin rpy="${pi/2} ${0} ${0}" xyz="${0} ${0} ${0.01605}"/>
-    <limit effort="100" velocity="10" />
+    <limit effort="5" velocity="1" />
     <!--<limit effort="100" lower="${-2*pi}" upper="${2*pi}" velocity="10" />-->
   </joint>
@@ -371,5 +371,5 @@
     <child link="clamp1"/>
     <origin rpy="${0} ${0} ${0}" xyz="${0} ${0} ${0.0235}"/>
-    <limit effort="100" velocity="10" />
+    <limit effort="5" velocity="1" />
     <!--<limit effort="100" lower="${-2*pi}" upper="${2*pi}" velocity="10" />-->
   </joint>
@@ -420,14 +420,14 @@
     <origin rpy="${0} ${pi/2} ${pi/2}" xyz="${0} ${0.016} ${0.022}"/>
   </joint>
-  <xacro:property name="tube1_mass" value="0.02035752" />
+  <xacro:property name="tube1_mass" value="0.039207076" />
   <xacro:property name="tube1_cog_x" value="0" />
   <xacro:property name="tube1_cog_y" value="0" />
   <xacro:property name="tube1_cog_z" value="0.3" />
-  <xacro:property name="tube1_ixx" value="0.002443367" />
+  <xacro:property name="tube1_ixx" value="${uc_inertia*4705.682308}" />
   <xacro:property name="tube1_ixy" value="0" />
   <xacro:property name="tube1_ixz" value="0" />
-  <xacro:property name="tube1_iyy" value="0.002443367" />
+  <xacro:property name="tube1_iyy" value="${uc_inertia*4705.682308}" />
   <xacro:property name="tube1_iyz" value="0" />
-  <xacro:property name="tube1_izz" value="0.000000929" />
+  <xacro:property name="tube1_izz" value="${uc_inertia*1.666300743}" />
     <link name="tube1">
       <visual>
@@ -456,14 +456,14 @@
       <origin rpy="${0} ${0} ${0}" xyz="${0} ${0} ${0.6}"/>
     </joint>
-    <xacro:property name="tip_mass" value="0.001658447" />
+    <xacro:property name="tip_mass" value="0.001540637" />
     <xacro:property name="tip_cog_x" value="0" />
     <xacro:property name="tip_cog_y" value="0" />
-    <xacro:property name="tip_cog_z" value="0.000163952" />
-    <xacro:property name="tip_ixx" value="${0.031944763*uc_inertia}" />
+    <xacro:property name="tip_cog_z" value="0.000367659054" />
+    <xacro:property name="tip_ixx" value="${0.028658362*uc_inertia}" />
     <xacro:property name="tip_ixy" value="${0*uc_inertia}" />
     <xacro:property name="tip_ixz" value="${0*uc_inertia}" />
-    <xacro:property name="tip_iyy" value="${0.031944763*uc_inertia}" />
+    <xacro:property name="tip_iyy" value="${0.028658362*uc_inertia}" />
     <xacro:property name="tip_iyz" value="${0*uc_inertia}" />
-    <xacro:property name="tip_izz" value="${0.033720057*uc_inertia}" />
+    <xacro:property name="tip_izz" value="${0.029110752*uc_inertia}" />
     <link name="tip">
       <visual>
