Commit message: created and sparated materials

File: src/fourth_model.urdf.xacro (robot description, xacro)
@@ -1,24 +1,8 @@
 <?xml version="1.0"?>
 <robot name="arm" xmlns:xacro="http://ros.org/wiki/xacro">
-    <!--<selfCollide>true</selfCollide>-->
-  <!-- Material and Colors-->
-  <material name="black">
-    <color rgba="${0/255} ${0/255} ${0/255} 1"/>
-  </material>
-  <material name="dark_grey">
-    <color rgba="${105/255} ${105/255} ${105/255} 1"/>
-  </material>
-  <material name="grey">
-    <color rgba="${128/255} ${128/255} ${128/255} 1"/>
-  </material>
-  <material name="light_grey">
-    <color rgba="${221/255} ${221/255} ${221/255} 1"/>
-  </material>
-  <material name="white">
-    <color rgba="${255/255} ${255/255} ${255/255} 1"/>
-  </material>
-  <material name="red">
-    <color rgba="${255/255} ${0/255} ${0/255} 1"/>
-  </material>
+    <!-- Import all Gazebo-customization elements, including Gazebo colors -->
+    <xacro:include filename="$(find mav_arm_force_controlled)/src/arm_gazebo_materials.gazebo" />
+    <!-- Import Rviz colors -->
+    <xacro:include filename="$(find mav_arm_force_controlled)/src/arm_rviz_materials.xacro" />
     <!-- General Variables-->
     <xacro:property name="pi" value="3.1415926535897931" />
@@ -49,7 +33,7 @@
     <!-- Mesh files are in mm. All mesh files are scaled by the factor 1000-->
     <xacro:property name="mesh_scale" value="0.001" />
-    <!-- Unit conversion for inertia from kg*mm² to kg m² -->
+    <!-- Unit conversion for inertia from kg*mm² to kg*m² -->
     <xacro:property name="uc_inertia" value="0.000001" />
-    <!-- The Mass and inertia elements are defined before the link element-->
+    <!-- The mass and inertia elements are defined before the link element -->
     <xacro:property name="baseplate_mass" value="0.034534697" />
     <xacro:property name="baseplate_cog_x" value="-0.0155840153" />
@@ -75,5 +59,4 @@
         </geometry>
       <origin rpy="0 0 0" xyz="0 0 0"/>
-       <material name="black"/>
     </visual>
     <collision>
@@ -437,5 +420,4 @@
         </geometry>
         <origin rpy="0 0 0" xyz="0 0 0"/>
-        <material name="black"/>
       </visual>
       <collision>
@@ -473,5 +455,4 @@
         </geometry>
         <origin rpy="0 0 0" xyz="0 0 0"/>
-        <material name="white"/>
       </visual>
       <collision>
@@ -487,42 +468,3 @@
       </inertial>
     </link>
-    <gazebo>
-      <plugin name="gazebo_ros_control" filename="libgazebo_ros_control.so">
-        <robotNamespace>/arm</robotNamespace>
-        <robotSimType>gazebo_ros_control/DefaultRobotHWSim</robotSimType>
-      </plugin>
-    </gazebo>
-    <gazebo reference="baseplate">
-      <selfCollide>true</selfCollide>
-    </gazebo>
-    <gazebo reference="actuator3">
-      <selfCollide>true</selfCollide>
-    </gazebo>
-    <gazebo reference="dynamixel_to_hebi">
-      <selfCollide>true</selfCollide>
-    </gazebo>
-    <gazebo reference="actuator2">
-      <selfCollide>true</selfCollide>
-    </gazebo>
-    <gazebo reference="clamp2">
-      <selfCollide>true</selfCollide>
-    </gazebo>
-    <gazebo reference="tube2">
-      <selfCollide>true</selfCollide>
-    </gazebo>
-    <gazebo reference="tube_adapter">
-      <selfCollide>true</selfCollide>
-    </gazebo>
-    <gazebo reference="actuator1">
-      <selfCollide>true</selfCollide>
-    </gazebo>
-    <gazebo reference="clamp1">
-      <selfCollide>true</selfCollide>
-    </gazebo>
-    <gazebo reference="tube1">
-      <selfCollide>true</selfCollide>
-    </gazebo>
-    <gazebo reference="tip">
-      <selfCollide>true</selfCollide>
-    </gazebo>
 </robot>

Commit message: adjusted topics

File: src/fourth_model.urdf.xacro (robot description, xacro)
@@ -179,5 +179,4 @@
       </geometry>
       <origin rpy="0 0 0" xyz="0 0 0"/>
-      <material name="red"/>
     </visual>
     <collision>

Commit message: added rviz launch file and adusted angle of assembly

File: src/fourth_model.urdf.xacro (robot description, xacro)
@@ -41,6 +41,6 @@
     <xacro:property name="baseplate_cog_z" value="0.01488134446" />
     <xacro:property name="baseplate_ixx" value="${60.4589042*uc_inertia}" />
-    <xacro:property name="baseplate_ixy" value="${-23.91373491*uc_inertia}" />
-    <xacro:property name="baseplate_ixz" value="${-9.415308277*uc_inertia}" />
+    <xacro:property name="baseplate_ixy" value="${0}" />
+    <xacro:property name="baseplate_ixz" value="${0}" />
     <xacro:property name="baseplate_iyy" value="${32.25701807*uc_inertia}" />
     <xacro:property name="baseplate_iyz" value="${17.84460765*uc_inertia}" />
@@ -112,7 +112,7 @@
     <parent link="actuator3"/>
     <child link="dynamixel_to_hebi"/>
-    <origin rpy="0 0 ${pi/2}" xyz="0 0 ${0.0235+0.012}"/>
+    <origin rpy="0 0 ${pi/2+pi/4}" xyz="0 0 ${0.0235+0.012}"/>
     <!--<limit effort="100" velocity="10"/>-->
-    <limit effort="5" lower="${-pi/2}" upper="${pi/2}" velocity="1" />
+    <limit effort="5" lower="${-3*pi/4}" upper="${pi/4}" velocity="1" />
   </joint>
   <transmission name="actuator3_dynamixel_trans">
@@ -132,7 +132,7 @@
   <xacro:property name="bearing_ixx" value="${139.5553029*uc_inertia}" />
   <xacro:property name="bearing_ixy" value="${0.414376963*uc_inertia}" />
-  <xacro:property name="bearing_ixz" value="${-31.92210758*uc_inertia}" />
+  <xacro:property name="bearing_ixz" value="${0}" />
   <xacro:property name="bearing_iyy" value="${162.416508*uc_inertia}" />
-  <xacro:property name="bearing_iyz" value="${-0.344517543*uc_inertia}" />
+  <xacro:property name="bearing_iyz" value="${0}" />
   <xacro:property name="bearing_izz" value="${80.76641832*uc_inertia}" />
   <link name="dynamixel_to_hebi">
@@ -179,4 +179,5 @@
       </geometry>
       <origin rpy="0 0 0" xyz="0 0 0"/>
+      <material name="red"/>
     </visual>
     <collision>
@@ -196,5 +197,5 @@
     <parent link="actuator2"/>
     <child link="clamp2"/>
-    <origin rpy="${pi/2} ${0} ${0}" xyz="${0} ${0} ${0.01605}"/>
+    <origin rpy="${pi/2} ${0} ${-pi/4}" xyz="${0} ${0} ${0.01605}"/>
     <limit effort="5" velocity="1" />
     <!--<limit effort="100" lower="${-2*pi}" upper="${2*pi}" velocity="10" />-->
@@ -214,8 +215,8 @@
   <xacro:property name="clamp2_cog_z" value="-0.01350332735" />
   <xacro:property name="clamp2_ixx" value="${21.61924342*uc_inertia}" />
-  <xacro:property name="clamp2_ixy" value="${-0.000002107*uc_inertia}" />
+  <xacro:property name="clamp2_ixy" value="${0}" />
   <xacro:property name="clamp2_ixz" value="${0.000000228*uc_inertia}" />
   <xacro:property name="clamp2_iyy" value="${23.46303475*uc_inertia}" />
-  <xacro:property name="clamp2_iyz" value="${-4.826007788*uc_inertia}" />
+  <xacro:property name="clamp2_iyz" value="${0}" />
   <xacro:property name="clamp2_izz" value="${7.990509672*uc_inertia}" />
   <link name="clamp2">
@@ -286,8 +287,8 @@
     <xacro:property name="clamp2_cog_z" value="20" />
     <xacro:property name="clamp2_ixx" value="${21.61924342*uc_inertia}" />
-    <xacro:property name="clamp2_ixy" value="${-0.000002107*uc_inertia}" />
+    <xacro:property name="clamp2_ixy" value="${0}" />
     <xacro:property name="clamp2_ixz" value="${0.000000228*uc_inertia}" />
     <xacro:property name="clamp2_iyy" value="${23.46303475*uc_inertia}" />
-    <xacro:property name="clamp2_iyz" value="${-4.826007788*uc_inertia}" />
+    <xacro:property name="clamp2_iyz" value="${0}" />
     <xacro:property name="clamp2_izz" value="${7.990509672*uc_inertia}" />
     <link name="tube_adapter">
@@ -352,5 +353,5 @@
     <parent link="actuator1"/>
     <child link="clamp1"/>
-    <origin rpy="${0} ${0} ${0}" xyz="${0} ${0} ${0.0235}"/>
+    <origin rpy="${0} ${0} ${pi/4}" xyz="${0} ${0} ${0.0235}"/>
     <limit effort="5" velocity="1" />
     <!--<limit effort="100" lower="${-2*pi}" upper="${2*pi}" velocity="10" />-->
@@ -371,6 +372,6 @@
   <xacro:property name="clamp1_cog_z" value="0.007840028704" />
   <xacro:property name="clamp1_ixx" value="${35.98639204*uc_inertia}" />
-  <xacro:property name="clamp1_ixy" value="${-0.036707373*uc_inertia}" />
-  <xacro:property name="clamp1_ixz" value="${-0.00032096*uc_inertia}" />
+  <xacro:property name="clamp1_ixy" value="${0}" />
+  <xacro:property name="clamp1_ixz" value="${0}" />
   <xacro:property name="clamp1_iyy" value="${26.23411723*uc_inertia}" />
   <xacro:property name="clamp1_iyz" value="${7.078559572*uc_inertia}" />

Commit message: changed to assembly form

File: src/fourth_model.urdf.xacro (robot description, xacro)
@@ -353,5 +353,5 @@
     <parent link="actuator1"/>
     <child link="clamp1"/>
-    <origin rpy="${0} ${0} ${pi/4}" xyz="${0} ${0} ${0.0235}"/>
+    <origin rpy="${0} ${0} ${-pi/4}" xyz="${0} ${0} ${0.0235}"/>
     <limit effort="5" velocity="1" />
     <!--<limit effort="100" lower="${-2*pi}" upper="${2*pi}" velocity="10" />-->

Commit message: small changes

File: src/fourth_model.urdf.xacro (robot description, xacro)
@@ -197,5 +197,5 @@
     <parent link="actuator2"/>
     <child link="clamp2"/>
-    <origin rpy="${pi/2} ${0} ${-pi/4}" xyz="${0} ${0} ${0.01605}"/>
+    <origin rpy="${pi/2} ${0} ${-pi/4-pi/8}" xyz="${0} ${0} ${0.01605}"/>
     <limit effort="5" velocity="1" />
     <!--<limit effort="100" lower="${-2*pi}" upper="${2*pi}" velocity="10" />-->
